File: kop3_onboarding/Hardware/Project#1/Project#1/Project#1.kicad_sch (KiCad schematic)
At the start: 0 parts

Commit message: Project #1 Complete
Created a simple led circuit using KiCad software. Created a schematic and a subsequent pcb layout.
Parts:
- added D1: LED_RED, layout:LED_0603_Symbol_on_F.SilkS, symbol Device:LED
- added J1: Conn_01x02, Connector_Molex:Molex_KK-254_AE-6410-02A_1x02_P2.54mm_Vertical, symbol Connector_Generic:Conn_01x02
- added R1: 105, Resistor_SMD:R_0603_1608Metric_Pad0.98x0.95mm_HandSolder, symbol device:R_US
- added SW1: SW_Push, Button_Switch_SMD:SW_DIP_SPSTx01_Slide_6.7x4.1mm_W8.61mm_P2.54mm_LowProfile, symbol Switch:SW_Push
Connections:
- new net: R1.1, SW1.2
- new net: D1.2 (A), R1.2
- new net +3V3: J1.2 (Pin_2), SW1.1
- new net GND: D1.1 (K), J1.1 (Pin_1)
Other:
- title: Template -> LED Project
