File: Hardware/Dev/proj2/proj2.kicad_pcb (KiCad board)
At the start: 2 copper layers, 0 parts

Commit message: made the jankiest board ever
Parts:
- added C1: .1uF, Capacitor_SMD:C_0603_1608Metric_Pad1.08x0.95mm_HandSolder, F.Cu at (145.1, 99.0)
- added C2: 0.1uF, Capacitor_SMD:C_0603_1608Metric_Pad1.08x0.95mm_HandSolder, F.Cu at (145.1, 104.8)
- added C3: 0.1uF, Capacitor_SMD:C_0603_1608Metric_Pad1.08x0.95mm_HandSolder, F.Cu at (145.1, 107.3)
- added C4: 0.1uF, Capacitor_SMD:C_0603_1608Metric_Pad1.08x0.95mm_HandSolder, F.Cu at (145.1, 109.8)
- added C5: 1uF, Capacitor_SMD:C_0603_1608Metric_Pad1.08x0.95mm_HandSolder, F.Cu at (145.1, 112.3)
- added C6: 1uF, Capacitor_SMD:C_0603_1608Metric_Pad1.08x0.95mm_HandSolder, F.Cu at (145.1, 114.8)
- added C7: 10uF, Capacitor_SMD:C_0603_1608Metric_Pad1.08x0.95mm_HandSolder, F.Cu at (145.1, 117.3)
- added C8: 1uF, Capacitor_SMD:C_0603_1608Metric_Pad1.08x0.95mm_HandSolder, F.Cu at (145.1, 119.8)
- added C9: 100uF, Capacitor_SMD:C_0603_1608Metric_Pad1.08x0.95mm_HandSolder, F.Cu at (145.1, 122.3)
- added D1: SM4003, Diode_SMD:D_MELF, F.Cu at (110.7, 186.4)
- added F1: Fuse, Fuse:Fuse_2512_6332Metric_Pad1.52x3.35mm_HandSolder, F.Cu at (151.5, 118.4)
- added J1: Conn_01x03, Connector_Molex:Molex_CLIK-Mate_502382-0370_1x03-1MP_P1.25mm_Vertical, F.Cu at (136.2, 100.3)
- added J2: Conn_01x02, Connector_Molex:Molex_CLIK-Mate_502382-0270_1x02-1MP_P1.25mm_Vertical, F.Cu at (153.5, 99.3)
- added J3: Conn_01x02, Connector_Molex:Molex_CLIK-Mate_502382-0270_1x02-1MP_P1.25mm_Vertical, F.Cu at (142.6, 129.2)
- added J4: Conn_01x02, Connector_Molex:Molex_CLIK-Mate_502382-0270_1x02-1MP_P1.25mm_Vertical, F.Cu at (150.9, 129.3)
- added Q1: FDMC8032L, Package_SON:Fairchild_DualPower33-6_3x3mm, F.Cu at (214.4, 154.4)
- added R1: 1000, Resistor_SMD:R_0201_0603Metric_Pad0.64x0.40mm_HandSolder, F.Cu at (141.4, 99.0)
Routing:
- net +24V: track 0.00 -> 94.8 mm
- net GND: track 0.00 -> 37.7 mm, vias 0 -> 2
- net /HORN_IN: track 0.00 -> 12.2 mm
- net /HORN_CTRL: track 0.00 -> 11.9 mm
- net Net-(J3-Pin_1): track 0.00 -> 11.6 mm
- net Net-(Q1B-D2): track 0.00 -> 8.29 mm
- net Net-(J2-Pin_1): track 0.00 -> 5.72 mm
- net Net-(C1-Pad1): track 0.00 -> 2.45 mm
- added copper zone on F.Cu, net +24V
- added copper zone on B.Cu, net GND
Other:
- board outline added: 29.8 x 42.8 mm
