File: Prog1/Prog1.kicad_pcb (KiCad board)
At the start: 2 copper layers, 0 parts

Commit message: led
Parts:
- added D1: LED, layout:LED_0603_Symbol_on_F.SilkS, F.Cu at (81.0, 66.5)
- added J1: Conn_01x02, Connector_Molex:Molex_CLIK-Mate_502382-0270_1x02-1MP_P1.25mm_Vertical, F.Cu at (70.5, 73.5)
- added R1: R, Resistor_SMD:R_0201_0603Metric_Pad0.64x0.40mm_HandSolder, F.Cu at (87.9, 67.5)
- added SW1: SW_Push, Button_Switch_SMD:SW_DIP_SPSTx01_Slide_6.7x4.1mm_W8.61mm_P2.54mm_LowProfile, F.Cu at (83.4, 75.5)
