File: Hardware/krp__Horns_v1.0/krp__Horns_v1.0.kicad_pcb (KiCad board)
At the start: 2 copper layers, 0 parts

Commit message: Finshed Horn onboarding project all flags resolved
Parts:
- added C1: 0.1uF, Capacitor_SMD:C_0201_0603Metric, F.Cu at (128.7, 84.2)
- added C2: 0.1uF, Capacitor_SMD:C_0201_0603Metric, F.Cu at (106.7, 78.5)
- added C3: 0.1uF, Capacitor_SMD:C_0201_0603Metric, F.Cu at (106.7, 80.8)
- added C4: 0.1uF, Capacitor_SMD:C_0201_0603Metric, F.Cu at (106.7, 83.2)
- added C5: 1uF, Capacitor_SMD:C_0201_0603Metric, F.Cu at (109.2, 77.2)
- added C6: 1uF, Capacitor_SMD:C_0201_0603Metric, F.Cu at (109.2, 79.8)
- added C7: 100uF, Capacitor_SMD:C_0201_0603Metric, F.Cu at (109.2, 82.4)
- added D1: D, Diode_SMD:D_0201_0603Metric, F.Cu at (125.5, 65.8)
- added F1: 2A, Fuse:Fuse_0402_1005Metric, F.Cu at (125.5, 74.0)
- added J1: Conn_01x02 (Horn Out), Connector_Molex:Molex_KK-254_AE-6410-02A_1x02_P2.54mm_Vertical, F.Cu at (121.5, 71.0)
- added J2: Conn_01x03 (Power), Connector_Molex:Molex_KK-396_5273-03A_1x03_P3.96mm_Vertical, F.Cu at (107.5, 71.0)
- added J3: Conn_01x02 (Horn Control), Connector_Molex:Molex_KK-254_AE-6410-02A_1x02_P2.54mm_Vertical, F.Cu at (114.5, 79.2)
- added J4: Conn_01x02 (Horn Out), Connector_Molex:Molex_KK-254_AE-6410-02A_1x02_P2.54mm_Vertical, F.Cu at (128.5, 68.5)
- added Q1: Q_NMOS_GDS, layout:TO-252-2, F.Cu at (127.4, 78.5)
- added R1: 1k, Resistor_SMD:R_0603_1608Metric_Pad0.98x0.95mm_HandSolder, F.Cu at (123.5, 83.0)
Routing:
- net GND: track 0.00 -> 61.8 mm, vias 0 -> 2
- net +24V: track 0.00 -> 21.5 mm
- net Net Label: track 0.00 -> 9.97 mm
- net Net-(C1-Pad1): track 0.00 -> 8.49 mm
- net Net-(J1-Pin_2): track 0.00 -> 8.05 mm
- net Net-(J1-Pin_1): track 0.00 -> 5.75 mm
- net Net-(Q1-D): track 0.00 -> 5.69 mm
- net Net-(D1-K): track 0.00 -> 5.01 mm
- net Net-(Q1-S): track 0.00 -> 2.72 mm
- added copper zone on F.Cu, net +24V
Other:
- board outline added: 30 x 22 mm
