File: Hardware/hornsprog/hornsprog.kicad_pcb (KiCad board)
At the start: 2 copper layers, 0 parts

Commit message: Updated Hardware Project
Parts:
- added C1: .1uF, Capacitor_SMD:C_0603_1608Metric, F.Cu at (130.1, 88.5)
- added C2: .1uF, Capacitor_SMD:C_0603_1608Metric, F.Cu at (126.9, 105.7)
- added C3: .1uF, Capacitor_SMD:C_0603_1608Metric, F.Cu at (122.2, 99.7)
- added C4: .1uF, Capacitor_SMD:C_0603_1608Metric, F.Cu at (122.2, 92.1)
- added C5: 1uF, Capacitor_SMD:C_0603_1608Metric, F.Cu at (122.2, 84.5)
- added C6: 1uF, Capacitor_SMD:C_0603_1608Metric, F.Cu at (122.2, 77.4)
- added C7: 10uF, Capacitor_SMD:C_0603_1608Metric, F.Cu at (122.2, 70.3)
- added C8: 10uF, Capacitor_SMD:C_0603_1608Metric, F.Cu at (122.2, 62.7)
- added C9: 100uF, Capacitor_SMD:C_0603_1608Metric, F.Cu at (122.2, 55.1)
- added D1: ES2DA-13-F, Diode_THT:D_DO-41_SOD81_P10.16mm_Horizontal, F.Cu at (138.3, 68.5)
- added HornControl1: Conn_01x02, Connector_Molex:Molex_KK-254_AE-6410-02A_1x02_P2.54mm_Vertical, F.Cu at (143.7, 103.3)
- added J1: Conn_01x03, Connector_Molex:Molex_KK-254_AE-6410-03A_1x03_P2.54mm_Vertical, F.Cu at (153.8, 92.0)
- added J3: Conn_01x02, Connector_Molex:Molex_KK-254_AE-6410-02A_1x02_P2.54mm_Vertical, F.Cu at (136.2, 54.5)
- added J4: Conn_01x02, Connector_Molex:Molex_KK-254_AE-6410-02A_1x02_P2.54mm_Vertical, F.Cu at (148.9, 57.0)
- added Q1: Q_NMOS_GDS, layout:TO-252-2, F.Cu at (142.1, 79.6)
- added R1: 1k Ohm, Resistor_SMD:R_0603_1608Metric, F.Cu at (144.2, 90.3)
- added REF**: MountingHole_3.2mm_M3, MountingHole:MountingHole_3.2mm_M3, F.Cu at (161.8, 50.6)
- added REF**: MountingHole_3.2mm_M3, MountingHole:MountingHole_3.2mm_M3, F.Cu at (118.5, 111.1)
Routing:
- net Net-(HornControl1-Pin_2): track 0.00 -> 299.2 mm
- net Net-(J1-Pin_2): track 0.00 -> 126.8 mm
- net /HORN_IN: track 0.00 -> 36.3 mm
- net Net-(Q1-G): track 0.00 -> 30.6 mm
- net /Horn Control: track 0.00 -> 13.2 mm
- net Net-(D1-A): track 0.00 -> 12.9 mm
- added copper zone on F.Cu, net /HORN_IN
Other:
- board outline added: 55.1 x 72.1 mm
