File: Hardware/hornsprog/hornsprog.kicad_sch (KiCad schematic)
At the start: 0 parts

Commit message: Advanced Hardware Project
Completed schematic for advanced hardware project.
Parts:
- added C1, C2, C3, C4: .1uF, Capacitor_SMD:C_0603_1608Metric, symbol device:C_Small
- added C5, C6: 1uF, Capacitor_SMD:C_0603_1608Metric, symbol device:C_Small
- added C7, C8: 10uF, Capacitor_SMD:C_0603_1608Metric, symbol device:C_Small
- added C9: 100uF, Capacitor_SMD:C_0603_1608Metric, symbol Device:C_Polarized_Small_US
- added D1: ES2DA-13-F, Diode_THT:D_DO-41_SOD81_P10.16mm_Horizontal, symbol Diode:1N4003
- added HornControl1, J3, J4: Conn_01x02, Connector_Molex:Molex_KK-254_AE-6410-02A_1x02_P2.54mm_Vertical, symbol Connector_Generic:Conn_01x02
- added J1: Conn_01x03, Connector_Molex:Molex_KK-254_AE-6410-03A_1x03_P2.54mm_Vertical, symbol Connector_Generic:Conn_01x03
- added Q1: Q_NMOS_GDS, layout:TO-252-2, symbol Device:Q_NMOS_GDS
- added R1: 1k Ohm, Resistor_SMD:R_0603_1608Metric, symbol device:R_US
Connections:
- new net: C2.1, C3.1, C4.1, C5.1, C6.1, C7.1, C8.1, C9.1, J1.2 (Pin_2), J4.1 (Pin_1)
- new net: C1.2, C2.2, C3.2, C4.2, C5.2, C6.2, C7.2, C8.2, C9.2, HornControl1.2 (Pin_2), J3.2 (Pin_2), Q1.3 (S)
- new net: C1.1, Q1.1 (G), R1.2
- new net: D1.2 (A), Q1.2 (D)
- new net HORN_IN: D1.1 (K), J3.1 (Pin_1), J4.2 (Pin_2)
- new net Horn Control: HornControl1.1 (Pin_1), R1.1

Commit message: Updated Hardware Project
Other:
- title: Template -> Horn Board Schematic
