File: Hardware/Horns/Horns_v2.0.kicad_sch (KiCad schematic)
At the start: 17 parts, among them J1 Conn_01x03, J2 Conn_01x02, J3 Conn_01x02, J4 Conn_01x02, Q1 Q_NMOS_GDS

Commit message: Horns done
Parts:
- C1, C2, C3, C4: footprint Capacitor_SMD:C_1210_3225Metric -> Capacitor_SMD:C_1206_3216Metric; MPN C1210H104J1GACTU -> GMC31X7R104K6R3NT
- C5, C6: footprint Capacitor_SMD:C_0201_0603Metric -> Capacitor_SMD:C_1206_3216Metric; MPN GRM033R60G105MEA2-03 -> C1206S105M9RAC7210
- C7, C8: footprint Capacitor_SMD:C_1206_3216Metric -> Capacitor_SMD:C_0805_2012Metric; MPN GMT31X7R106K25NT2 -> GMC21X6S106K6R3NT
- C9: footprint Capacitor_SMD:CP_Elec_6.3x7.7 -> Capacitor_SMD:CP_Elec_6.3x5.4_Nichicon; MPN UWT1V101MCL1GS -> UWT0G101MCL1GB
- renumbered J3 to HORN_1, J4 to HORN_2
Connections:
- net GND: now also C2.1, C3.1, C4.1, C5.1, C6.1, C7.1, C8.1, C9.1, Q1.3 (S); no longer C2.2, C3.2, C4.2, C5.2, C6.2, C7.2, C8.2, C9.2, J1.1 (Pin_1)
- new net: C2.2, C3.2, C4.2, C5.2, C6.2, C7.2, C8.2, C9.2, J1.1 (Pin_1)
