File: Hardware/jkim_Horns_v1.0./jkim_Horns_v1.0..kicad_pcb (KiCad board)
At the start: 2 copper layers, 0 parts

Commit message: Working on pcb
Parts:
- added C1: 0.1 µF, Capacitor_SMD:C_0603_1608Metric, F.Cu at (61.5, 73.0)
- added C2: 100 µF, Capacitor_SMD:C_0603_1608Metric, F.Cu at (79.5, 62.3)
- added C3: 10 µF, Capacitor_SMD:C_0603_1608Metric, F.Cu at (82.7, 67.5)
- added C4: 10 µF, Capacitor_SMD:C_0603_1608Metric, F.Cu at (83.2, 71.5)
- added C5: 1 µF, Capacitor_SMD:C_0603_1608Metric, F.Cu at (95.0, 67.7)
- added C6: 1 µF, Capacitor_SMD:C_0603_1608Metric, F.Cu at (90.5, 72.2)
- added C7: 0.1 µF, Capacitor_SMD:C_0603_1608Metric, F.Cu at (89.7, 80.0)
- added C8: 0.1 µF, Capacitor_SMD:C_0603_1608Metric, F.Cu at (83.7, 75.5)
- added C9: 0.1 µF, Capacitor_SMD:C_0603_1608Metric, F.Cu at (75.2, 75.5)
- added D1: D, Diode_SMD:D_0603_1608Metric_Pad1.05x0.95mm_HandSolder, F.Cu at (71.0, 75.0)
- added F2: 2A, Diode_SMD:D_SOD-123F, F.Cu at (67.0, 75.0)
- added J1: Conn_01x03, Connector_Molex:Molex_KK-254_AE-6410-03A_1x03_P2.54mm_Vertical, F.Cu at (61.5, 64.5)
- added J2: Conn_01x02, Connector_Molex:Molex_KK-254_AE-6410-02A_1x02_P2.54mm_Vertical, F.Cu at (56.0, 69.0)
- added J3: Conn_01x02, Connector_Molex:Molex_KK-254_AE-6410-02A_1x02_P2.54mm_Vertical, F.Cu at (70.5, 85.0)
- added J4: Conn_01x02, Connector_Molex:Molex_KK-254_AE-6410-02A_1x02_P2.54mm_Vertical, F.Cu at (64.0, 85.0)
- added Q1: Q_NMOS_DGS, Package_TO_SOT_SMD:TO-252-2, F.Cu at (58.0, 77.5)
- added R1: 1 kΩ, Resistor_SMD:R_0603_1608Metric_Pad0.98x0.95mm_HandSolder, F.Cu at (61.6, 70.0)
- added REF**: MountingHole_3.2mm_M3, MountingHole:MountingHole_3.2mm_M3, F.Cu at (76.0, 85.0)
- added REF**: MountingHole_3.2mm_M3, MountingHole:MountingHole_3.2mm_M3, F.Cu at (56.0, 63.5)
- added REF**: MountingHole_3.2mm_M3, MountingHole:MountingHole_3.2mm_M3, F.Cu at (56.0, 86.0)
- added REF**: MountingHole_3.2mm_M3, MountingHole:MountingHole_3.2mm_M3, F.Cu at (87.5, 59.5)

Commit message: working on layout
Parts:
- moved C5 29.6 mm to (65.5, 69.5), turned to 0 degrees
- moved C6 25.3 mm to (65.2, 72.5), turned to 0 degrees
- moved C7 21.9 mm to (69.0, 72.8), turned to 90 degrees
- moved REF** 15.4 mm to (72.5, 63.0)
- moved C4 14.9 mm to (68.5, 69.3), turned to -90 degrees
- moved C8 12.0 mm to (72.0, 72.8), turned to 90 degrees
- moved C3 10.9 mm to (72.0, 69.3), turned to -90 degrees
- moved J3 8.72 mm to (72.5, 76.5), turned to -90 degrees
- moved C2 8.32 mm to (75.0, 69.3), turned to -90 degrees
- moved D1 7.53 mm to (66.0, 80.6)
- moved REF** 3.64 mm to (72.5, 86.0)
- moved C9 2.73 mm to (75.0, 72.8), turned to 90 degrees
- moved J4 2.10 mm to (64.5, 87.0), turned to 90 degrees
- moved F2 1.49 mm to (66.5, 76.4)
- moved J1 1.00 mm to (61.5, 63.5)

Commit message: Finished layout
Parts:
- moved C7 2.14 mm to (67.0, 72.0), turned to -90 degrees
- moved C8 2.14 mm to (70.0, 72.0), turned to -90 degrees
- moved C9 2.14 mm to (73.0, 72.0), turned to -90 degrees
- moved C2 2.07 mm to (73.0, 68.7)
- moved C3 2.07 mm to (70.0, 68.7)
- moved C5 1.97 mm to (64.2, 68.0), turned to 180 degrees
- moved C6 1.79 mm to (64.2, 71.0), turned to 180 degrees
- moved C4 1.58 mm to (67.0, 68.8)
- moved R1 1.54 mm to (60.5, 68.9), turned to -90 degrees
- moved J3 1.46 mm to (71.2, 75.8)
- moved C1 1.24 mm to (60.5, 72.3), turned to -90 degrees
- moved REF** 1.00 mm to (56.0, 62.5), turned to 180 degrees
- moved REF** 0.71 mm to (72.0, 86.5)
- moved REF** 0.71 mm to (72.0, 62.5), turned to 180 degrees
- moved REF** 0.50 mm to (56.0, 86.5)
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Routing:
- net Net-(J3-Pin_1): track 0.00 -> 25.8 mm
- net +24V: track 0.00 -> 24.7 mm
- net GND: track 0.00 -> 19.2 mm
- net Net-(J3-Pin_2): track 0.00 -> 12.1 mm
- net Net-(Q1-D): track 0.00 -> 6.71 mm
- net /HORN_CTL: track 0.00 -> 6.00 mm
- net Net-(J2-Pin_1): track 0.00 -> 4.91 mm
- net Net-(D1-K): track 0.00 -> 3.62 mm
- net /HORN_IN: track 0.00 -> 2.30 mm
- net Net-(C1-Pad1): track 0.00 -> 1.67 mm
- added copper zone on F.Cu, net +24V
- added copper zone on B.Cu, net GND
Other:
- board outline added: 24 x 32 mm
