File: Hardware/Horns Board Project/HornsBoard_v1.kicad_pcb (KiCad board)
At the start: 2 copper layers, 0 parts

Commit message: Horns Bord PCB
Parts:
- added C1: 0.1uF, Capacitor_SMD:C_0201_0603Metric_Pad0.64x0.40mm_HandSolder, F.Cu at (178.0, 126.6)
- added C2: 100uF, Capacitor_SMD:C_0603_1608Metric_Pad1.08x0.95mm_HandSolder, F.Cu at (166.5, 129.8)
- added C3: 1uF, Capacitor_SMD:C_0201_0603Metric_Pad0.64x0.40mm_HandSolder, F.Cu at (174.2, 117.7)
- added C4: 1uF, Capacitor_SMD:C_0201_0603Metric_Pad0.64x0.40mm_HandSolder, F.Cu at (163.7, 130.9)
- added C5: 0.1uF, Capacitor_SMD:C_0201_0603Metric_Pad0.64x0.40mm_HandSolder, F.Cu at (176.5, 124.6)
- added C6: 0.1uF, Capacitor_SMD:C_0201_0603Metric_Pad0.64x0.40mm_HandSolder, F.Cu at (163.7, 128.3)
- added C7: 0.1uF, Capacitor_SMD:C_0201_0603Metric_Pad0.64x0.40mm_HandSolder, F.Cu at (170.5, 117.8)
- added D1: D_Small, Diode_SMD:D_0603_1608Metric_Pad1.05x0.95mm_HandSolder, F.Cu at (166.5, 132.8)
- added F1: 2A, Fuse:Fuse_0603_1608Metric_Pad1.05x0.95mm_HandSolder, F.Cu at (180.8, 126.6)
- added J1: Conn_01x03, Connector_Molex:Molex_KK-254_AE-6410-03A_1x03_P2.54mm_Vertical, F.Cu at (166.1, 119.3)
- added J2: Conn_01x02, Connector_Molex:Molex_KK-254_AE-6410-02A_1x02_P2.54mm_Vertical, F.Cu at (178.0, 119.5)
- added J3: Conn_01x02, Connector_Molex:Molex_KK-254_AE-6410-02A_1x02_P2.54mm_Vertical, F.Cu at (170.5, 131.0)
- added J4: Conn_01x02, Connector_Molex:Molex_KK-254_AE-6410-02A_1x02_P2.54mm_Vertical, F.Cu at (179.8, 131.0)
- added Q1: Q_NMOS_DGS, Transistor_Power:GaN_Systems_GaNPX-3_5x6.6mm_Drain2.93x0.6mm, F.Cu at (172.6, 122.2)
- added R1: 1000, Resistor_SMD:R_0201_0603Metric_Pad0.64x0.40mm_HandSolder, F.Cu at (179.7, 124.6)
- added REF**: MountingHole_3.2mm_M3, MountingHole:MountingHole_3.2mm_M3, F.Cu at (186.0, 119.0)
- added REF**: MountingHole_3.2mm_M3, MountingHole:MountingHole_3.2mm_M3, F.Cu at (159.0, 119.0)
- added REF**: MountingHole_3.2mm_M3, MountingHole:MountingHole_3.2mm_M3, F.Cu at (186.0, 131.0)
- added REF**: MountingHole_3.2mm_M3, MountingHole:MountingHole_3.2mm_M3, F.Cu at (159.0, 131.0)
Routing:
- net GND: track 0.00 -> 39.4 mm
- net /HORN_IN: track 0.00 -> 31.7 mm
- net Net-(Q1-G): track 0.00 -> 17.4 mm
- net +24V: track 0.00 -> 14.3 mm
- net /HORN_CTRL: track 0.00 -> 5.86 mm
- added copper zone on F.Cu, net +24V
- added copper zone on B.Cu, net GND
Other:
- board outline added: 35 x 20 mm

Commit message: Horns Board PCB
Parts:
- added C8: 10uf, Capacitor_SMD:C_0603_1608Metric_Pad1.08x0.95mm_HandSolder, F.Cu at (165.4, 124.9)
- added C9: 10uF, Capacitor_SMD:C_0603_1608Metric_Pad1.08x0.95mm_HandSolder, F.Cu at (167.4, 126.6)
- C1, C3, C4, C5, C6, C7: footprint Capacitor_SMD:C_0201_0603Metric_Pad0.64x0.40mm_HandSolder -> Capacitor_SMD:C_0603_1608Metric_Pad1.08x0.95mm_HandSolder
- D1: footprint Diode_SMD:D_0603_1608Metric_Pad1.05x0.95mm_HandSolder -> Diode_SMD:D_0402_1005Metric_Pad0.77x0.64mm_HandSolder
- R1: footprint Resistor_SMD:R_0201_0603Metric_Pad0.64x0.40mm_HandSolder -> Resistor_SMD:R_0402_1005Metric_Pad0.72x0.64mm_HandSolder
- moved J1 2.27 mm to (165.9, 117.1)
- moved C7 1.47 mm to (171.2, 116.5)
- moved C4 1.30 mm to (164.3, 132.1), turned to 180 degrees
- moved F1 1.11 mm to (182.0, 126.6)
- moved D1 1.07 mm to (166.8, 133.8)
- moved REF** 1.00 mm to (187.0, 119.0)
- moved REF** 1.00 mm to (187.0, 131.0)
- moved R1 0.84 mm to (180.4, 125.0)
- moved C5 0.78 mm to (177.3, 124.8)
- moved C3 0.68 mm to (174.6, 117.1)
- moved J2 0.21 mm to (178.1, 119.3)
- moved C2 0.17 mm to (166.6, 129.9), turned to 0 degrees
- moved C6 0.13 mm to (163.8, 128.3), turned to 180 degrees
Routing:
- net +24V: track 14.3 -> 74.0 mm
- net GND: track 39.4 -> 65.2 mm
- net Net-(Q1-G): track 17.4 -> 20.4 mm
Other:
- board size 35 x 20 mm -> 36 x 20 mm
