File: Hardware/horns/horns.kicad_pcb (KiCad board)
At the start: 2 copper layers, 0 parts

Commit message: pcb layout done
Parts:
- added C10: 0u1, Capacitor_SMD:C_0805_2012Metric, F.Cu at (129.9, 77.0)
- added C2: 1u, Capacitor_SMD:C_0805_2012Metric, F.Cu at (120.0, 103.0)
- added C3: 1u, Capacitor_SMD:C_0805_2012Metric, F.Cu at (117.0, 103.0)
- added C4: 0u1, Capacitor_SMD:C_0805_2012Metric, F.Cu at (114.0, 102.0)
- added C5: 0u1, Capacitor_SMD:C_0805_2012Metric, F.Cu at (112.0, 99.0)
- added C6: 0u1, Capacitor_SMD:C_0805_2012Metric, F.Cu at (111.0, 96.0)
- added C7: 10u, Capacitor_SMD:C_0805_2012Metric, F.Cu at (111.0, 93.0)
- added C8-C4: 10u, Capacitor_SMD:C_0805_2012Metric, F.Cu at (111.0, 90.0)
- added C9: 100u, layout:CP_Oval_L16.0mm_W8.0mm_P11.5mm, F.Cu at (122.0, 94.0)
- added D2: ES2DA-13-F, Diode_SMD:D_SMA, F.Cu at (124.0, 78.0)
- added F1: 2A, layout:Fuse_Littelfuse_1206, F.Cu at (120.0, 76.6)
- added J1: PWR_IN, Connector_Molex:Molex_KK-254_AE-6410-03A_1x03_P2.54mm_Vertical, F.Cu at (125.0, 86.0)
- added J2: Horn_Control, Connector_Molex:Molex_KK-254_AE-6410-02A_1x02_P2.54mm_Vertical, F.Cu at (132.0, 70.0)
- added J3: horn_out_1, Connector_Molex:Molex_KK-254_AE-6410-02A_1x02_P2.54mm_Vertical, F.Cu at (113.0, 77.0)
- added J4: horn_out_2, Connector_Molex:Molex_KK-254_AE-6410-02A_1x02_P2.54mm_Vertical, F.Cu at (114.0, 85.5)
- added Q1: IRFR010PBF, layout:TO-252-2, F.Cu at (122.0, 68.1)
- added R2: 1k, Resistor_SMD:R_0603_1608Metric_Pad0.98x0.95mm_HandSolder, F.Cu at (127.0, 75.9)
- added REF**: MountingHole_3.2mm_M3, MountingHole:MountingHole_3.2mm_M3, F.Cu at (113.0, 67.0)
- added REF**: MountingHole_3.2mm_M3, MountingHole:MountingHole_3.2mm_M3, F.Cu at (130.0, 102.0)
Routing:
- net Net-(D2-A): track 0.00 -> 9.70 mm
- net /HORNS_CTRL: track 0.00 -> 9.33 mm
- net Net-(J3-Pin_1): track 0.00 -> 6.41 mm
- net /HORN_IN: track 0.00 -> 3.02 mm
- net Net-(C10-Pad2): track 0.00 -> 2.09 mm
- net GND: vias 0 -> 9
- added copper zone on F.Cu, net +24V
- added copper zone on B.Cu, net GND
Other:
- board outline added: 27 x 46 mm
