File: Hardware/horns/horns.kicad_sch (KiCad schematic)
At the start: 17 parts, among them J1 PWR_IN, J2 Horn_Control, J3 horn_out_1, J4 horn_out_2, Q1 IRFR010PBF

Commit message: footprints assigned (idk if they right doh), pcb meta data added (my name)
Parts:
- C1, C2, C3, C4, C5, C6, C7, C8: footprint (none) -> Capacitor_SMD:C_0805_2012Metric
- C9: footprint (none) -> layout:CP_Oval_L16.0mm_W8.0mm_P11.5mm
- D1: footprint (none) -> Diode_SMD:D_SMA
- F1: footprint (none) -> layout:Fuse_Littelfuse_1206
- J1: footprint Connector_Molex:Molex_KK-254_AE-6410-03A_1x03_P2.54mm_Vertical -> layout:Molex_KK-254_1x03_P2.54mm_Horizontal
- J2, J3, J4: footprint Connector_Molex:Molex_KK-254_AE-6410-02A_1x02_P2.54mm_Vertical -> layout:Molex_KK-254_1x02_P2.54mm_Horizontal
- Q1: footprint (none) -> layout:TO-252-2
Changed lines of the file:
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@@
 			)
 		)
-		(property "Footprint" ""
+		(property "Footprint" "layout:TO-252-2"
 			(at 180.34 82.55 0)
 			(effects
@@
 			)
 		)
-		(property "Footprint" ""
+		(property "Footprint" "Capacitor_SMD:C_0805_2012Metric"
 			(at 132.08 140.0048 0)
 			(effects
@@
 			)
 		)
-		(property "Footprint" "Connector_Molex:Molex_KK-254_AE-6410-03A_1x03_P2.54mm_Vertical"
+		(property "Footprint" "layout:Molex_KK-254_1x03_P2.54mm_Horizontal"
 			(at 113.03 97.79 0)
 			(effects
@@
 			)
 		)
-		(property "Footprint" "Connector_Molex:Molex_KK-254_AE-6410-02A_1x02_P2.54mm_Vertical"
+		(property "Footprint" "layout:Molex_KK-254_1x02_P2.54mm_Horizontal"
 			(at 129.54 71.12 0)
 			(effects
@@
 			)
 		)
-		(property "Footprint" ""
+		(property "Footprint" "Capacitor_SMD:C_0805_2012Metric"
 			(at 132.08 129.8448 0)
 			(effects
@@
 			)
 		)
-		(property "Footprint" ""
+		(property "Footprint" "layout:CP_Oval_L16.0mm_W8.0mm_P11.5mm"
 			(at 132.08 145.0848 0)
 			(effects
@@
 			)
 		)
-		(property "Footprint" ""
+		(property "Footprint" "Diode_SMD:D_SMA"
 			(at 142.24 86.36 0)
 			(effects
@@
 			)
 		)
-		(property "Datasheet" "~"
+		(property "Datasheet" "https://www.diodes.com/assets/Datasheets/ds14002.pdf"
 			(at 142.24 86.36 0)
 			(effects
@@
 			)
 		)
-		(property "Footprint" ""
+		(property "Footprint" "layout:Fuse_Littelfuse_1206"
 			(at 160.02 80.518 90)
 			(effects
@@
 			)
 		)
-		(property "Footprint" "Connector_Molex:Molex_KK-254_AE-6410-02A_1x02_P2.54mm_Vertical"
+		(property "Footprint" "layout:Molex_KK-254_1x02_P2.54mm_Horizontal"
 			(at 153.67 110.49 0)
 			(effects
@@
 			)
 		)
-		(property "Footprint" ""
+		(property "Footprint" "Capacitor_SMD:C_0805_2012Metric"
 			(at 132.08 134.9248 0)
 			(effects
@@
 			)
 		)
-		(property "Footprint" "Connector_Molex:Molex_KK-254_AE-6410-02A_1x02_P2.54mm_Vertical"
+		(property "Footprint" "layout:Molex_KK-254_1x02_P2.54mm_Horizontal"
 			(at 149.86 71.12 0)
 			(effects
@@
 			)
 		)
-		(property "Footprint" ""
+		(property "Footprint" "Capacitor_SMD:C_0805_2012Metric"
 			(at 132.08 119.6848 0)
 			(effects
@@
 			)
 		)
-		(property "Footprint" ""
+		(property "Footprint" "Capacitor_SMD:C_0805_2012Metric"
 			(at 162.2552 128.27 0)
 			(effects
@@
 			)
 		)
-		(property "Footprint" ""
+		(property "Footprint" "Capacitor_SMD:C_0805_2012Metric"
 			(at 132.08 114.6048 0)
 			(effects
@@
 			)
 		)
-		(property "Footprint" ""
+		(property "Footprint" "Capacitor_SMD:C_0805_2012Metric"
 			(at 132.08 109.5248 0)
 			(effects
@@
 			)
 		)
-		(property "Footprint" ""
+		(property "Footprint" "Capacitor_SMD:C_0805_2012Metric"
 			(at 132.08 124.7648 0)
 			(effects

Commit message: pcb layout done
Parts:
- removed C1: 0u1, Capacitor_SMD:C_0805_2012Metric, symbol Device:C
- removed D1: ES2DA-13-F, Diode_SMD:D_SMA, symbol Device:D
- removed R1: 1k, Resistor_SMD:R_0603_1608Metric_Pad0.98x0.95mm_HandSolder, symbol device:R
- added C10: 0u1, Capacitor_SMD:C_0805_2012Metric, symbol Device:C
- added D2: ES2DA-13-F, Diode_SMD:D_SMA, symbol Device:D
- added R2: 1k, Resistor_SMD:R_0603_1608Metric_Pad0.98x0.95mm_HandSolder, symbol device:R
Connections:
- net +24V: now also D2.1 (K)
- net GND: now also J2.1 (Pin_1), C10.1
- net HORNS_CTRL: now also R2.1
- net HORN_IN: now also F1.2, Q1.1 (D); no longer F1.1, J3.2 (Pin_2)
- new net: D2.2 (A), F1.1, J3.2 (Pin_2)
- new net: C10.2, R2.2

Commit message: completed horns changes and added gerber/dfm
Parts:
- J1: footprint layout:Molex_KK-254_1x03_P2.54mm_Horizontal -> Connector_Molex:Molex_Micro-Fit_3.0_43650-0300_1x03_P3.00mm_Horizontal
- J2, J3, J4: footprint layout:Molex_KK-254_1x02_P2.54mm_Horizontal -> Connector_Molex:Molex_Micro-Fit_3.0_43650-0200_1x02_P3.00mm_Horizontal
Changed lines of the file:
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@@
 			)
 		)
-		(property "Footprint" "layout:Molex_KK-254_1x03_P2.54mm_Horizontal"
+		(property "Footprint" "Connector_Molex:Molex_Micro-Fit_3.0_43650-0300_1x03_P3.00mm_Horizontal"
 			(at 113.03 97.79 0)
 			(effects
@@
 			)
 		)
-		(property "Footprint" "layout:Molex_KK-254_1x02_P2.54mm_Horizontal"
+		(property "Footprint" "Connector_Molex:Molex_Micro-Fit_3.0_43650-0200_1x02_P3.00mm_Horizontal"
 			(at 129.54 71.12 0)
 			(effects
@@
 			)
 		)
-		(property "Footprint" "layout:Molex_KK-254_1x02_P2.54mm_Horizontal"
+		(property "Footprint" "Connector_Molex:Molex_Micro-Fit_3.0_43650-0200_1x02_P3.00mm_Horizontal"
 			(at 153.67 110.49 0)
 			(effects
@@
 			)
 		)
-		(property "Footprint" "layout:Molex_KK-254_1x02_P2.54mm_Horizontal"
+		(property "Footprint" "Connector_Molex:Molex_Micro-Fit_3.0_43650-0200_1x02_P3.00mm_Horizontal"
 			(at 149.86 71.12 0)
 			(effects
