File: Hardware/prog1/prog1.kicad_pcb (KiCad board)
At the start: 2 copper layers, 0 parts

Commit message: LED project PCB
Parts:
- added D1: LED, layout:LED_0603_Symbol_on_F.SilkS, F.Cu at (124.0, 101.0)
- added J1: Conn, Connector_Molex:Molex_KK-254_AE-6410-02A_1x02_P2.54mm_Vertical, F.Cu at (125.5, 108.0)
- added R1: R_US, Resistor_SMD:R_0603_1608Metric_Pad0.98x0.95mm_HandSolder, F.Cu at (129.0, 101.0)
- added REF**: MountingHole, MountingHole:MountingHole_3.2mm_M3, F.Cu at (126.0, 96.0)
- added REF**: MountingHole, MountingHole:MountingHole_3.2mm_M3, F.Cu at (134.0, 108.0)
- added SW1: SW_Push, Button_Switch_SMD:SW_DIP_SPSTx01_Slide_6.7x4.1mm_W8.61mm_P2.54mm_LowProfile, F.Cu at (134.0, 98.0)
Routing:
- net Net-(R1-Pad1): track 0.00 -> 10.2 mm
- net Net-(D1-A): track 0.00 -> 8.53 mm
- net GND: track 0.00 -> 4.50 mm, vias 0 -> 1
- added copper zone on F.Cu, net +3V3
- added copper zone on B.Cu, net GND
Other:
- board outline added: 19 x 23 mm
