File: Hardware/Project2_HornsBoard/Project2_HornsBoard.kicad_sch (KiCad schematic)
At the start: 0 parts

Commit message: firmware project 2 complete
Parts:
- added C1: 1μ, symbol Device:C
- added C2, C3, C4: 0.1μF, symbol Device:C
- added C5, C6: 1μF, symbol Device:C
- added C7, C8: 10μF, symbol Device:C
- added C9: 100μF_Polarized, symbol Device:C_Polarized
- added D1: D, symbol Device:D
- added F1: 2A, symbol device:Fuse
- added J1: Power, Connector_Molex:Molex_KK-254_AE-6410-03A_1x03_P2.54mm_Vertical, symbol Connector_Generic:Conn_01x03
- added J2: HORN_CTL, Connector_Molex:Molex_KK-254_AE-6410-02A_1x02_P2.54mm_Vertical, symbol Connector_Generic:Conn_01x02
- added J3: HORN_OUT_A, Connector_Molex:Molex_KK-254_AE-6410-02A_1x02_P2.54mm_Vertical, symbol Connector_Generic:Conn_01x02
- added J4: HORN_OUT_B, Connector_Molex:Molex_KK-254_AE-6410-02A_1x02_P2.54mm_Vertical, symbol Connector_Generic:Conn_01x02
- added Q1: Q_NMOS_DGS, symbol device:Q_NMOS_DGS
- added R1: 1kΩ, Resistor_SMD:R_0603_1608Metric_Pad0.98x0.95mm_HandSolder, symbol Device:R_US
Connections:
- new net: D1.1 (K), J1.2 (Pin_2), J3.1 (Pin_1)
- new net: C1.2, J2.2 (Pin_2)
- new net: Q1.2 (G), R1.1
- new net: F1.1, Q1.1 (D)
- new net: J3.2 (Pin_2), J4.1 (Pin_1)
- new net: F1.2, J4.2 (Pin_2)
- new net +24V: C2.2, C3.2, C4.2, C5.2, C6.2, C7.2, C8.2, C9.1, D1.2 (A), J1.3 (Pin_3), Q1.3 (S)
- new net GND: C1.1, C2.1, C3.1, C4.1, C5.1, C6.1, C7.1, C8.1, C9.2, J1.1 (Pin_1)
- new net Net Label: J2.1 (Pin_1), R1.2
Other:
- title: Template -> Project2_HornsBoard
