File: Hardware/Dev/OnboardingHornsBoardv1.0/OnboardingHornsBoardv1.0.kicad_sch (KiCad schematic)
At the start: 0 parts

Commit message: Onboarding Horns Board PCB design
Parts:
- added C1, C2, C3, C4: 0.1uF, Capacitor_SMD:C_0603_1608Metric, symbol device:C
- added C10: 100uF, Capacitor_SMD:C_0603_1608Metric, symbol Device:C_Polarized_Small_US
- added C5, C6: 1uF, Capacitor_SMD:C_0603_1608Metric, symbol device:C
- added C7, C8: 10uF, Capacitor_SMD:C_0603_1608Metric, symbol device:C
- added D1: US2DA, Diode_SMD:D_SMA, symbol Diode:US2DA
- added F1: 2A, Fuse:Fuse_0402_1005Metric, symbol Device:Fuse
- added Horn1, Horn2, J3: Conn_01x02, Connector_Molex:Molex_CLIK-Mate_502382-0270_1x02-1MP_P1.25mm_Vertical, symbol Connector_Generic:Conn_01x02
- added J1: Conn_01x03, Connector_Molex:Molex_CLIK-Mate_502382-0370_1x03-1MP_P1.25mm_Vertical, symbol Connector_Generic:Conn_01x03
- added Q1: Q_NMOS_DGS, layout:TO-252-2, symbol Device:Q_NMOS_DGS
- added R1: 1k, Resistor_SMD:R_0201_0603Metric_Pad0.64x0.40mm_HandSolder, symbol Device:R
Connections:
- new net: D1.1 (K), Horn1.1 (Pin_1)
- new net: Horn1.2 (Pin_2), Horn2.1 (Pin_1)
- new net: F1.1, Horn2.2 (Pin_2)
- new net: F1.2, Q1.3 (S)
- new net: C1.1, J3.2 (Pin_2), R1.1
- new net +24V: C10.1, C2.1, C3.1, C4.1, C5.1, C6.1, C7.1, C8.1, D1.2 (A), J1.2 (Pin_2)
- new net GND: C1.2, C10.2, C2.2, C3.2, C4.2, C5.2, C6.2, C7.2, C8.2, J1.1 (Pin_1), J1.3 (Pin_3), Q1.1 (D), R1.2
- new net Horn Control: J3.1 (Pin_1), Q1.2 (G)
Other:
- title: Template -> Horns Board

Commit message: Horns Board Onboarding Project
Parts:
- R1: footprint Resistor_SMD:R_0201_0603Metric_Pad0.64x0.40mm_HandSolder -> Resistor_SMD:R_0603_1608Metric
Connections:
- net +24V: now also D1.1 (K), Horn1.1 (Pin_1); no longer D1.2 (A)
- net at F1.1, Horn2.2 (Pin_2): now also D1.2 (A)
Changed lines of the file:
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@@
+	)
+	(junction
+		(at 143.51 92.71)
+		(diameter 0)
+		(color 0 0 0 0)
 	)
 	(junction
@@
 	)
 	(junction
+		(at 172.72 92.71)
+		(diameter 0)
+		(color 0 0 0 0)
+	)
+	(junction
 		(at 228.6 120.65)
 		(diameter 0)
@@
 	(wire
 		(pts
-			(xy 149.86 96.52) (xy 166.37 96.52)
+			(xy 149.86 92.71) (xy 166.37 92.71)
 		)
 		(stroke
@@
 	(wire
 		(pts
+			(xy 134.62 92.71) (xy 134.62 96.52)
+		)
+		(stroke
+			(width 0)
+			(type default)
+		)
+	)
+	(wire
+		(pts
 			(xy 124.46 93.98) (xy 124.46 96.52)
 		)
@@
 	(wire
 		(pts
-			(xy 149.86 96.52) (xy 149.86 92.71)
-		)
-		(stroke
-			(width 0)
-			(type default)
-		)
-	)
-	(wire
-		(pts
 			(xy 140.97 99.06) (xy 140.97 100.33)
 		)
@@
 	(wire
 		(pts
-			(xy 168.91 92.71) (xy 204.47 92.71)
+			(xy 134.62 92.71) (xy 143.51 92.71)
+		)
+		(stroke
+			(width 0)
+			(type default)
+		)
+	)
+	(wire
+		(pts
+			(xy 143.51 92.71) (xy 147.32 92.71)
+		)
+		(stroke
+			(width 0)
+			(type default)
+		)
+	)
+	(wire
+		(pts
+			(xy 168.91 92.71) (xy 172.72 92.71)
 		)
 		(stroke
@@
 	(wire
 		(pts
+			(xy 172.72 96.52) (xy 161.29 96.52)
+		)
+		(stroke
+			(width 0)
+			(type default)
+		)
+	)
+	(wire
+		(pts
+			(xy 172.72 92.71) (xy 172.72 96.52)
+		)
+		(stroke
+			(width 0)
+			(type default)
+		)
+	)
+	(wire
+		(pts
 			(xy 124.46 96.52) (xy 120.65 96.52)
 		)
@@
 	(wire
 		(pts
+			(xy 153.67 96.52) (xy 143.51 96.52)
+		)
+		(stroke
+			(width 0)
+			(type default)
+		)
+	)
+	(wire
+		(pts
 			(xy 120.65 110.49) (xy 124.46 110.49)
 		)
@@
 	(wire
 		(pts
+			(xy 172.72 92.71) (xy 204.47 92.71)
+		)
+		(stroke
+			(width 0)
+			(type default)
+		)
+	)
+	(wire
+		(pts
 			(xy 243.84 120.65) (xy 252.73 120.65)
 		)
@@
 	(wire
 		(pts
+			(xy 143.51 96.52) (xy 143.51 92.71)
+		)
+		(stroke
+			(width 0)
+			(type default)
+		)
+	)
+	(wire
+		(pts
 			(xy 228.6 128.27) (xy 229.87 128.27)
 		)
@@
 	(wire
 		(pts
-			(xy 142.24 96.52) (xy 147.32 96.52)
-		)
-		(stroke
-			(width 0)
-			(type default)
-		)
-	)
-	(wire
-		(pts
 			(xy 148.59 106.68) (xy 160.02 106.68)
 		)
@@
 	(wire
 		(pts
-			(xy 147.32 96.52) (xy 147.32 92.71)
-		)
-		(stroke
-			(width 0)
-			(type default)
-		)
-	)
-	(wire
-		(pts
 			(xy 120.65 81.28) (xy 109.22 81.28)
 		)
@@
 		(pts
 			(xy 171.45 99.06) (xy 180.34 99.06)
-		)
-		(stroke
-			(width 0)
-			(type default)
-		)
-	)
-	(wire
-		(pts
-			(xy 166.37 96.52) (xy 166.37 92.71)
 		)
 		(stroke
@@
 	)
 	(symbol
-		(lib_id "Diode:US2DA")
-		(at 138.43 96.52 180)
-		(unit 1)
-		(exclude_from_sim no)
-		(in_bom yes)
-		(on_board yes)
-		(dnp no)
-		(fields_autoplaced yes)
-		(property "Reference" "D1"
-			(at 138.43 90.17 0)
-			(effects
-				(font
-					(size 1.27 1.27)
-				)
-			)
-		)
-		(property "Value" "US2DA"
-			(at 138.43 92.71 0)
-			(effects
-				(font
-					(size 1.27 1.27)
-				)
-			)
-		)
-		(property "Footprint" "Diode_SMD:D_SMA"
-			(at 138.43 92.075 0)
-			(effects
-				(font
-					(size 1.27 1.27)
-				)
-				(hide yes)
-			)
-		)
-		(property "Datasheet" "https://www.diodes.com/assets/Datasheets/ds14002.pdf"
-			(at 138.43 96.52 0)
-			(effects
-				(font
-					(size 1.27 1.27)
-				)
-				(hide yes)
-			)
-		)
-		(property "Description" "200V, 1.5A, General Purpose Rectifier Diode, SMA(DO-214AC)"
-			(at 138.43 96.52 0)
-			(effects
-				(font
-					(size 1.27 1.27)
-				)
-				(hide yes)
-			)
-		)
-		(pin "1"
-		)
-		(pin "2"
-		)
-		(instances
-			(project ""
-				(path "/1e1b062d-fad0-427c-a622-c5b8a80b5268"
-					(reference "D1")
-					(unit 1)
-				)
-			)
-		)
-	)
-	(symbol
 		(lib_id "power:PWR_FLAG")
 		(at 124.46 93.98 270)
@@
 	)
 	(symbol
+		(lib_id "Diode:US2DA")
+		(at 157.48 96.52 0)
+		(unit 1)
+		(exclude_from_sim no)
+		(in_bom yes)
+		(on_board yes)
+		(dnp no)
+		(fields_autoplaced yes)
+		(property "Reference" "D1"
+			(at 157.48 90.17 0)
+			(effects
+				(font
+					(size 1.27 1.27)
+				)
+			)
+		)
+		(property "Value" "US2DA"
+			(at 157.48 92.71 0)
+			(effects
+				(font
+					(size 1.27 1.27)
+				)
+			)
+		)
+		(property "Footprint" "Diode_SMD:D_SMA"
+			(at 157.48 100.965 0)
+			(effects
+				(font
+					(size 1.27 1.27)
+				)
+				(hide yes)
+			)
+		)
+		(property "Datasheet" "https://www.diodes.com/assets/Datasheets/ds14002.pdf"
+			(at 157.48 96.52 0)
+			(effects
+				(font
+					(size 1.27 1.27)
+				)
+				(hide yes)
+			)
+		)
+		(property "Description" "200V, 1.5A, General Purpose Rectifier Diode, SMA(DO-214AC)"
+			(at 157.48 96.52 0)
+			(effects
+				(font
+					(size 1.27 1.27)
+				)
+				(hide yes)
+			)
+		)
+		(pin "1"
+		)
+		(pin "2"
+		)
+		(instances
+			(project "OnboardingHornsBoardv1.0"
+				(path "/1e1b062d-fad0-427c-a622-c5b8a80b5268"
+					(reference "D1")
+					(unit 1)
+				)
+			)
+		)
+	)
+	(symbol
 		(lib_id "device:C")
 		(at 171.45 102.87 0)
@@
 			)
 		)
-		(property "Footprint" "Resistor_SMD:R_0201_0603Metric_Pad0.64x0.40mm_HandSolder"
+		(property "Footprint" "Resistor_SMD:R_0603_1608Metric"
 			(at 232.41 122.428 90)
 			(effects

Commit message: re-added unsaved changes
Parts:
- Horn1, Horn2, J3: footprint Connector_Molex:Molex_CLIK-Mate_502382-0270_1x02-1MP_P1.25mm_Vertical -> Connector_Molex:Molex_Micro-Fit_3.0_43650-0200_1x02_P3.00mm_Horizontal
- J1: footprint Connector_Molex:Molex_CLIK-Mate_502382-0370_1x03-1MP_P1.25mm_Vertical -> Connector_Molex:Molex_Micro-Fit_3.0_43650-0300_1x03_P3.00mm_Horizontal
Changed lines of the file:
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@@
 			)
 		)
-		(property "Footprint" "Connector_Molex:Molex_CLIK-Mate_502382-0270_1x02-1MP_P1.25mm_Vertical"
+		(property "Footprint" "Connector_Molex:Molex_Micro-Fit_3.0_43650-0200_1x02_P3.00mm_Horizontal"
 			(at 147.32 87.63 0)
 			(effects
@@
 			)
 		)
-		(property "Footprint" "Connector_Molex:Molex_CLIK-Mate_502382-0370_1x03-1MP_P1.25mm_Vertical"
+		(property "Footprint" "Connector_Molex:Molex_Micro-Fit_3.0_43650-0300_1x03_P3.00mm_Horizontal"
 			(at 115.57 96.52 0)
 			(effects
@@
 			)
 		)
-		(property "Footprint" "Connector_Molex:Molex_CLIK-Mate_502382-0270_1x02-1MP_P1.25mm_Vertical"
+		(property "Footprint" "Connector_Molex:Molex_Micro-Fit_3.0_43650-0200_1x02_P3.00mm_Horizontal"
 			(at 166.37 87.63 0)
 			(effects
@@
 			)
 		)
-		(property "Footprint" "Connector_Molex:Molex_CLIK-Mate_502382-0270_1x02-1MP_P1.25mm_Vertical"
+		(property "Footprint" "Connector_Molex:Molex_Micro-Fit_3.0_43650-0200_1x02_P3.00mm_Horizontal"
 			(at 233.68 105.41 0)
 			(effects
