File: Hardware/Dev/Horns Board/Hornsboard.kicad_pcb (KiCad board)
At the start: 2 copper layers, 0 parts

Commit message: Very Challenged Circuits
Parts:
- added C1: 0.1 uF, Capacitor_SMD:C_0603_1608Metric_Pad1.08x0.95mm_HandSolder, F.Cu at (137.4, 71.5)
- added C2: 0.1 uF, Capacitor_SMD:C_0603_1608Metric_Pad1.08x0.95mm_HandSolder, F.Cu at (137.4, 74.5)
- added C3: 0.1 uF, Capacitor_SMD:C_0603_1608Metric_Pad1.08x0.95mm_HandSolder, F.Cu at (137.4, 78.0)
- added C4: 0.1 uF, Capacitor_SMD:C_0603_1608Metric_Pad1.08x0.95mm_HandSolder, F.Cu at (137.4, 82.0)
- added C5: 1 uF, Capacitor_SMD:C_0603_1608Metric_Pad1.08x0.95mm_HandSolder, F.Cu at (137.4, 85.5)
- added C6: 1 uF, Capacitor_SMD:C_0603_1608Metric_Pad1.08x0.95mm_HandSolder, F.Cu at (137.4, 89.0)
- added C7: 10 uF, Capacitor_SMD:C_0603_1608Metric_Pad1.08x0.95mm_HandSolder, F.Cu at (142.9, 71.5)
- added C8: 10 uF, Capacitor_SMD:C_0603_1608Metric_Pad1.08x0.95mm_HandSolder, F.Cu at (142.9, 74.5)
- added C9: 100 uF, Capacitor_SMD:C_0603_1608Metric_Pad1.08x0.95mm_HandSolder, F.Cu at (142.9, 78.0)
- added D1: LED, LED_SMD:LED_0603_1608Metric_Pad1.05x0.95mm_HandSolder, F.Cu at (144.9, 85.5)
- added F1: 2A, Fuse:Fuse_0603_1608Metric, F.Cu at (145.8, 90.0)
- added J1: Conn_01x03, Connector_Molex:Molex_Micro-Fit_3.0_43650-0300_1x03_P3.00mm_Horizontal, F.Cu at (152.0, 77.4)
- added J2: Horns_out2, Connector_Molex:Molex_Micro-Fit_3.0_43650-0200_1x02_P3.00mm_Horizontal, F.Cu at (126.0, 66.0)
- added J3: Horn Control, Connector_Molex:Molex_Micro-Fit_3.0_43650-0200_1x02_P3.00mm_Horizontal, F.Cu at (117.0, 77.8)
- added J4: Horns_out1, Connector_Molex:Molex_Micro-Fit_3.0_43650-0200_1x02_P3.00mm_Horizontal, F.Cu at (128.5, 88.3)
- added Q1: Q_NMOS_GDS, layout:TO-252-2, F.Cu at (141.4, 61.5)
- added R1: 1000 Ohm, Resistor_SMD:R_0603_1608Metric_Pad0.98x0.95mm_HandSolder, F.Cu at (144.9, 82.0)
- added REF**: MountingHole_3.2mm_M3, MountingHole:MountingHole_3.2mm_M3, F.Cu at (154.5, 61.5)
- added REF**: MountingHole_3.2mm_M3, MountingHole:MountingHole_3.2mm_M3, F.Cu at (154.5, 88.0)
- added REF**: MountingHole_3.2mm_M3, MountingHole:MountingHole_3.2mm_M3, F.Cu at (117.0, 88.0)
- added REF**: MountingHole_3.2mm_M3, MountingHole:MountingHole_3.2mm_M3, F.Cu at (117.0, 60.5)
Routing:
- net Net-(D1-K): track 0.00 -> 50.9 mm
- net +24V: track 0.00 -> 46.7 mm, vias 0 -> 2
- net /Horn Control I guess: track 0.00 -> 46.0 mm, vias 0 -> 2
- net Net-(J2-Pin_1): track 0.00 -> 37.8 mm, vias 0 -> 2
- net Net-(Q1-D): track 0.00 -> 31.6 mm, vias 0 -> 2
- net Net-(Q1-G): track 0.00 -> 31.3 mm
- net Net-(J2-Pin_2): track 0.00 -> 22.9 mm
- net Net-(D1-A): track 0.00 -> 21.0 mm, vias 0 -> 2
- net GND: track 0.00 -> 10.4 mm, vias 0 -> 4
- added copper zone on F.Cu, net +24V
- added copper zone on B.Cu, net GND
Other:
- board outline added: 51 x 36.5 mm
