File: Hardware/Dev/Horns Board/Hornsboard.kicad_sch (KiCad schematic)
At the start: 0 parts

Commit message: Challenged Hardware Project
Parts:
- added C1, C2, C3, C4: 0.1 uF, symbol Device:C
- added C5, C6: 1 uF, symbol Device:C
- added C7, C8: 10 uF, symbol Device:C
- added C9: 100 uF, symbol Device:C
- added D1: LED, symbol Device:LED
- added F1: 2A, symbol device:Fuse
- added J1: Conn_01x03, symbol Connector_Generic:Conn_01x03
- added J2: Horns_out2, symbol Connector_Generic:Conn_01x02
- added J3: Horn Control, symbol Connector_Generic:Conn_01x02
- added J4: Horns_out1, symbol Connector_Generic:Conn_01x02
- added Q1: BUZ11, Package_TO_SOT_THT:TO-220-3_Vertical, symbol Transistor_FET:BUZ11
- added R1: 1000 Ohm, symbol device:R_US
Connections:
- new net: C1.2, Q1.1 (G), R1.2
- new net: F1.2, J2.1 (Pin_1)
- new net: J2.2 (Pin_2), J4.1 (Pin_1)
- new net: C2.1, C3.1, C4.1, C5.1, C6.1, C7.1, C8.1, C9.1, D1.1 (K), J1.2 (Pin_2)
- new net: D1.2 (A), J4.2 (Pin_2)
- new net: F1.1, Q1.2 (D)
- new net +24V: C2.2, C3.2, C4.2, C5.2, C6.2, C7.2, C8.2, C9.2
- new net GND: J1.1 (Pin_1), J1.3 (Pin_3), J3.2 (Pin_2), Q1.3 (S)
- new net Horn Control I guess: C1.1, J3.1 (Pin_1), R1.1

Commit message: Very Challenged Circuits
Parts:
- removed Q1: BUZ11, Package_TO_SOT_THT:TO-220-3_Vertical, symbol Transistor_FET:BUZ11
- added Q1: Q_NMOS_GDS, layout:TO-252-2, symbol device:Q_NMOS_GDS
- C1, C2, C3, C4, C5, C6, C7, C8, C9: footprint (none) -> Capacitor_SMD:C_0603_1608Metric_Pad1.08x0.95mm_HandSolder
- D1: footprint (none) -> LED_SMD:LED_0603_1608Metric_Pad1.05x0.95mm_HandSolder
- F1: footprint (none) -> Fuse:Fuse_0603_1608Metric
- J1: footprint (none) -> Connector_Molex:Molex_Micro-Fit_3.0_43650-0300_1x03_P3.00mm_Horizontal
- J2, J3, J4: footprint (none) -> Connector_Molex:Molex_Micro-Fit_3.0_43650-0200_1x02_P3.00mm_Horizontal
- R1: footprint (none) -> Resistor_SMD:R_0603_1608Metric_Pad0.98x0.95mm_HandSolder
Connections:
- net GND: now also Q1.3 (S)
- net at C1.2, R1.2: now also Q1.1 (G)
- net at F1.1: now also Q1.2 (D)
Other:
- moved on the sheet: C2, C3, C4, C5, C6, C7, C8, C9
