File: Hardware/Prog1/prog1_v1.kicad_pcb (KiCad board)
At the start: 2 copper layers, 16 x 25 mm, 6 parts, among them SW1 SW_Push

Commit message: integrated feedback
Parts:
- removed Jr1: Conn_01x02, Connector_Molex:Molex_KK-254_AE-6410-02A_1x02_P2.54mm_Vertical
- added REF**: Molex_Micro-Fit_3.0_43650-0300_1x03_P3.00mm_Horizontal, Connector_Molex:Molex_Micro-Fit_3.0_43650-0300_1x03_P3.00mm_Horizontal, F.Cu at (134.3, 96.0)
- moved REF** 1.00 mm to (145.0, 100.0)
Other:
- board size 16 x 25 mm -> 32 x 24 mm
