File: Hardware/Dev/HornBoard_project2/HornBoard_project2_v0.0.kicad_sch (KiCad schematic)
At the start: 0 parts

Commit message: hardware project 2 schematic complete
Parts:
- added C1, C2, C3, C4: 0.1microF, symbol device:C
- added C5, C6: 1microF, symbol device:C
- added C7, C8: 10microF, symbol device:C
- added C9: C_Polarized, symbol device:C_Polarized
- added D1: 1N4003, Diode_THT:D_DO-41_SOD81_P10.16mm_Horizontal, symbol Diode:1N4003
- added F1: Fuse, symbol device:Fuse
- added J1: Power In, symbol Connector_Generic:Conn_01x03
- added J2: Horn Control, symbol Connector_Generic:Conn_01x02
- added J3: Horn Out 1, symbol Connector_Generic:Conn_01x02
- added J4: Horn Out 2, symbol Connector_Generic:Conn_01x02
- added Q1: Q_NMOS_GSD, symbol Device:Q_NMOS_GSD
- added R1: 1000ohms, symbol device:R_US
- added TP1, TP2, TP3: TestPoint, symbol Connector:TestPoint
Connections:
- new net: C1.2, Q1.1 (G), R1.2, TP2.1
- new net: D1.2 (A), Q1.2 (S), TP3.1
- new net: F1.1, J3.1 (Pin_1), J4.1 (Pin_1)
- new net: D1.1 (K), F1.2
- new net: J2.2 (Pin_2), R1.1
- new net GND: C1.1, C2.2, C3.2, C4.2, C5.2, C6.2, C7.2, C8.2, C9.2, J1.1 (Pin_1), J1.3 (Pin_3), J2.1 (Pin_1), Q1.3 (D)
- new net VCC: C2.1, C3.1, C4.1, C5.1, C6.1, C7.1, C8.1, C9.1, J1.2 (Pin_2), J3.2 (Pin_2), J4.2 (Pin_2), TP1.1
Other:
- title: Template -> Horn_Board

Commit message: update 10/1
Parts:
- C1, C2, C3, C4: footprint (none) -> Capacitor_SMD:C_0805_2012Metric
- C5, C6, C7, C8: footprint (none) -> Capacitor_SMD:C_0805_2012Metric_Pad1.18x1.45mm_HandSolder
- C9: footprint (none) -> Capacitor_SMD:CP_Elec_6.3x5.8
- F1: footprint (none) -> Fuse:Fuse_1206_3216Metric
- J1: footprint (none) -> Connector_Molex:Molex_CLIK-Mate_502382-0370_1x03-1MP_P1.25mm_Vertical
- J2, J3, J4: footprint (none) -> Connector_Molex:Molex_CLIK-Mate_502382-0270_1x02-1MP_P1.25mm_Vertical
- Q1: footprint (none) -> layout:TO-252-2
- R1: footprint (none) -> Resistor_SMD:R_0805_2012Metric
- TP1, TP2, TP3: footprint (none) -> TestPoint:TestPoint_Pad_D1.0mm
Connections:
- net VCC renamed +24V24
Changed lines of the file:
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@@
 			)
 		)
-		(property "Footprint" ""
+		(property "Footprint" "TestPoint:TestPoint_Pad_D1.0mm"
 			(at 49.53 45.72 0)
 			(effects
@@
 			)
 		)
-		(property "Footprint" ""
+		(property "Footprint" "Capacitor_SMD:C_0805_2012Metric_Pad1.18x1.45mm_HandSolder"
 			(at 195.2752 68.58 0)
 			(effects
@@
 			)
 		)
-		(property "Datasheet" "~"
+		(property "Datasheet" "https://docs.google.com/spreadsheets/d/1BsfQQcO9C6DZCsRaXUlFlo91Tg2WpOkGARC1WS5S8t0/edit?gid=619195040#gid=619195040"
 			(at 194.31 64.77 0)
 			(effects
@@
 			)
 		)
-		(property "Footprint" ""
+		(property "Footprint" "layout:TO-252-2"
 			(at 35.56 106.68 0)
 			(effects
@@
 			)
 		)
-		(property "Datasheet" "~"
+		(property "Datasheet" "http://www.infineon.com/cms/en/product/packages/PG-TO252/PG-TO252-3-1/"
 			(at 30.48 109.22 0)
 			(effects
@@
 			)
 		)
-		(property "Footprint" ""
+		(property "Footprint" "Capacitor_SMD:C_0805_2012Metric_Pad1.18x1.45mm_HandSolder"
 			(at 180.0352 68.58 0)
 			(effects
@@
 			)
 		)
-		(property "Datasheet" "~"
+		(property "Datasheet" "https://docs.google.com/spreadsheets/d/1BsfQQcO9C6DZCsRaXUlFlo91Tg2WpOkGARC1WS5S8t0/edit?gid=619195040#gid=619195040"
 			(at 179.07 64.77 0)
 			(effects
@@
 			)
 		)
-		(property "Footprint" ""
+		(property "Footprint" "Capacitor_SMD:C_0805_2012Metric_Pad1.18x1.45mm_HandSolder"
 			(at 211.7852 68.58 0)
 			(effects
@@
 			)
 		)
-		(property "Datasheet" "~"
+		(property "Datasheet" "https://docs.google.com/spreadsheets/d/1BsfQQcO9C6DZCsRaXUlFlo91Tg2WpOkGARC1WS5S8t0/edit?gid=619195040#gid=619195040"
 			(at 210.82 64.77 0)
 			(effects
@@
 			)
 		)
-		(property "Footprint" ""
+		(property "Footprint" "TestPoint:TestPoint_Pad_D1.0mm"
 			(at 33.02 118.11 0)
 			(effects
@@
 			)
 		)
-		(property "Footprint" ""
+		(property "Footprint" "Connector_Molex:Molex_CLIK-Mate_502382-0270_1x02-1MP_P1.25mm_Vertical"
 			(at 54.61 100.33 0)
 			(effects
@@
 			)
 		)
-		(property "Datasheet" "~"
+		(property "Datasheet" "http://www.molex.com/pdm_docs/sd/5023820270_sd.pdf"
 			(at 54.61 100.33 0)
 			(effects
@@
 			)
 		)
-		(property "Footprint" ""
+		(property "Footprint" "Capacitor_SMD:C_0805_2012Metric"
 			(at 16.2052 100.33 0)
 			(effects
@@
 			)
 		)
-		(property "Datasheet" "~"
+		(property "Datasheet" "https://docs.google.com/spreadsheets/d/1BsfQQcO9C6DZCsRaXUlFlo91Tg2WpOkGARC1WS5S8t0/edit?gid=619195040#gid=619195040"
 			(at 15.24 96.52 0)
 			(effects
@@
 			)
 		)
-		(property "Footprint" ""
+		(property "Footprint" "Connector_Molex:Molex_CLIK-Mate_502382-0270_1x02-1MP_P1.25mm_Vertical"
 			(at 54.61 82.55 0)
 			(effects
@@
 			)
 		)
-		(property "Datasheet" "~"
+		(property "Datasheet" "http://www.molex.com/pdm_docs/sd/5023820270_sd.pdf"
 			(at 54.61 82.55 0)
 			(effects
@@
 			)
 		)
-		(property "Footprint" ""
+		(property "Footprint" "TestPoint:TestPoint_Pad_D1.0mm"
 			(at 12.7 104.14 0)
 			(effects
@@
 			)
 		)
-		(property "Footprint" ""
+		(property "Footprint" "Capacitor_SMD:C_0805_2012Metric_Pad1.18x1.45mm_HandSolder"
 			(at 164.7952 68.58 0)
 			(effects
@@
 			)
 		)
-		(property "Datasheet" "~"
+		(property "Datasheet" "https://docs.google.com/spreadsheets/d/1BsfQQcO9C6DZCsRaXUlFlo91Tg2WpOkGARC1WS5S8t0/edit?gid=619195040#gid=619195040"
 			(at 163.83 64.77 0)
 			(effects
@@
 			)
 		)
-		(property "Footprint" ""
+		(property "Footprint" "Capacitor_SMD:C_0805_2012Metric"
 			(at 131.7752 68.58 0)
 			(effects
@@
 			)
 		)
-		(property "Datasheet" "~"
+		(property "Datasheet" "https://docs.google.com/spreadsheets/d/1BsfQQcO9C6DZCsRaXUlFlo91Tg2WpOkGARC1WS5S8t0/edit?gid=619195040#gid=619195040"
 			(at 130.81 64.77 0)
 			(effects
@@
 			)
 		)
-		(property "Footprint" ""
+		(property "Footprint" "Resistor_SMD:R_0805_2012Metric"
 			(at 26.416 95.504 90)
 			(effects
@@
 			)
 		)
-		(property "Datasheet" "~"
+		(property "Datasheet" "https://www.pcb-3d.com/wordpress/wp-content/uploads/ipc-sm-782a_amendment_1_and_2.pdf"
 			(at 25.4 95.25 0)
 			(effects
@@
 			)
 		)
-		(property "Footprint" ""
+		(property "Footprint" "Connector_Molex:Molex_CLIK-Mate_502382-0370_1x03-1MP_P1.25mm_Vertical"
 			(at 55.88 60.96 0)
 			(effects
@@
 			)
 		)
-		(property "Datasheet" "~"
+		(property "Datasheet" "http://www.molex.com/pdm_docs/sd/5023820270_sd.pdf"
 			(at 55.88 60.96 0)
 			(effects
@@
 			)
 		)
-		(property "Value" "VCC"
+		(property "Value" "+24V24"
 			(at 33.02 38.1 0)
 			(effects
@@
 			)
 		)
-		(property "Footprint" ""
+		(property "Footprint" "Fuse:Fuse_1206_3216Metric"
 			(at 35.052 113.03 90)
 			(effects
@@
 			)
 		)
-		(property "Datasheet" "~"
+		(property "Datasheet" "http://www.tortai-tech.com/upload/download/2011102023233369053.pdf"
 			(at 36.83 113.03 0)
 			(effects
@@
 			)
 		)
-		(property "Footprint" ""
+		(property "Footprint" "Connector_Molex:Molex_CLIK-Mate_502382-0270_1x02-1MP_P1.25mm_Vertical"
 			(at 57.15 116.84 0)
 			(effects
@@
 			)
 		)
-		(property "Datasheet" "~"
+		(property "Datasheet" "http://www.molex.com/pdm_docs/sd/5023820270_sd.pdf"
 			(at 57.15 116.84 0)
 			(effects
@@
 			)
 		)
-		(property "Footprint" ""
+		(property "Footprint" "Capacitor_SMD:C_0805_2012Metric"
 			(at 115.2652 68.58 0)
 			(effects
@@
 			)
 		)
-		(property "Datasheet" "~"
+		(property "Datasheet" "https://docs.google.com/spreadsheets/d/1BsfQQcO9C6DZCsRaXUlFlo91Tg2WpOkGARC1WS5S8t0/edit?gid=619195040#gid=619195040"
 			(at 114.3 64.77 0)
 			(effects
@@
 			)
 		)
-		(property "Footprint" ""
+		(property "Footprint" "Capacitor_SMD:CP_Elec_6.3x5.8"
 			(at 93.6752 68.58 0)
 			(effects
@@
 			)
 		)
-		(property "Footprint" ""
+		(property "Footprint" "Capacitor_SMD:C_0805_2012Metric"
 			(at 148.2852 68.58 0)
 			(effects
@@
 			)
 		)
-		(property "Datasheet" "~"
+		(property "Datasheet" "https://docs.google.com/spreadsheets/d/1BsfQQcO9C6DZCsRaXUlFlo91Tg2WpOkGARC1WS5S8t0/edit?gid=619195040#gid=619195040"
 			(at 147.32 64.77 0)
 			(effects
