File: Hardware/Dev/HornBoard_project2/HornBoard_project2_v0.0.kicad_pcb (KiCad board)
At the start: 2 copper layers, 0 parts

Commit message: update 10/1
Parts:
- added C1: 0.1microF, Capacitor_SMD:C_0805_2012Metric, F.Cu at (85.0, 36.0)
- added C2: 0.1microF, Capacitor_SMD:C_0805_2012Metric, F.Cu at (83.0, 42.0)
- added C3: 0.1microF, Capacitor_SMD:C_0805_2012Metric, F.Cu at (95.0, 53.0)
- added C4: 0.1microF, Capacitor_SMD:C_0805_2012Metric, F.Cu at (94.0, 60.0)
- added C5: 1microF, Capacitor_SMD:C_0805_2012Metric_Pad1.18x1.45mm_HandSolder, F.Cu at (90.0, 72.0)
- added C6: 1microF, Capacitor_SMD:C_0805_2012Metric_Pad1.18x1.45mm_HandSolder, F.Cu at (94.0, 82.0)
- added C7: 10microF, Capacitor_SMD:C_0805_2012Metric_Pad1.18x1.45mm_HandSolder, F.Cu at (78.0, 80.0)
- added C8: 10microF, Capacitor_SMD:C_0805_2012Metric_Pad1.18x1.45mm_HandSolder, F.Cu at (81.0, 88.0)
- added C9: C_Polarized, Capacitor_SMD:CP_Elec_6.3x5.8, F.Cu at (72.3, 62.0)
- added D1: 1N4003, Diode_THT:D_DO-41_SOD81_P10.16mm_Horizontal, F.Cu at (64.8, 43.0)
- added F1: Fuse, Fuse:Fuse_1206_3216Metric, F.Cu at (58.6, 43.0)
- added J1: Power In, Connector_Molex:Molex_CLIK-Mate_502382-0370_1x03-1MP_P1.25mm_Vertical, F.Cu at (50.0, 44.0)
- added J2: Horn Control, Connector_Molex:Molex_CLIK-Mate_502382-0270_1x02-1MP_P1.25mm_Vertical, F.Cu at (118.4, 33.0)
- added J3: Horn Out 1, Connector_Molex:Molex_CLIK-Mate_502382-0270_1x02-1MP_P1.25mm_Vertical, F.Cu at (136.0, 56.0)
- added J4: Horn Out 2, Connector_Molex:Molex_CLIK-Mate_502382-0270_1x02-1MP_P1.25mm_Vertical, F.Cu at (108.9, 45.5)
- added Q1: Q_NMOS_GSD, layout:TO-252-2, F.Cu at (52.2, 61.7)
- added R1: 1000ohms, Resistor_SMD:R_0805_2012Metric, F.Cu at (105.0, 76.0)
- added TP1: TestPoint, TestPoint:TestPoint_Pad_D1.0mm, F.Cu at (107.0, 62.0)
- added TP2: TestPoint, TestPoint:TestPoint_Pad_D1.0mm, F.Cu at (107.0, 93.0)
- added TP3: TestPoint, TestPoint:TestPoint_Pad_D1.0mm, F.Cu at (94.0, 95.0)

Commit message: hardware project 2 horn board submit
Parts:
- added REF**: MountingHole_3.2mm_M3, MountingHole:MountingHole_3.2mm_M3, F.Cu at (51.0, 34.0)
- added REF**: MountingHole_3.2mm_M3, MountingHole:MountingHole_3.2mm_M3, F.Cu at (51.0, 85.0)
- added REF**: MountingHole_3.2mm_M3, MountingHole:MountingHole_3.2mm_M3, F.Cu at (114.0, 85.0)
- added REF**: MountingHole_3.2mm_M3, MountingHole:MountingHole_3.2mm_M3, F.Cu at (114.0, 34.0)
- J1: footprint Connector_Molex:Molex_CLIK-Mate_502382-0370_1x03-1MP_P1.25mm_Vertical -> Connector_Molex:Molex_Micro-Fit_3.0_43650-0300_1x03_P3.00mm_Horizontal
- J2, J3, J4: footprint Connector_Molex:Molex_CLIK-Mate_502382-0270_1x02-1MP_P1.25mm_Vertical -> Connector_Molex:Molex_Micro-Fit_3.0_43650-0200_1x02_P3.00mm_Horizontal
- moved TP3 59.2 mm to (58.0, 48.0)
- moved TP2 41.4 mm to (101.0, 52.0)
- moved TP1 33.1 mm to (74.0, 65.0)
- moved J2 29.8 mm to (90.0, 42.0), turned to 180 degrees
- moved J3 24.3 mm to (112.0, 52.0), turned to 90 degrees
- moved R1 24.2 mm to (95.0, 54.0)
- moved C9 21.2 mm to (52.0, 56.0)
- moved C2 20.1 mm to (74.0, 60.0), turned to 90 degrees
- moved C1 18.1 mm to (83.0, 54.0), turned to 180 degrees
- moved Q1 18.0 mm to (67.2, 51.7)
- moved F1 15.4 mm to (74.0, 43.0)
- moved C3 13.4 mm to (83.0, 59.0), turned to -90 degrees
- moved C6 12.2 mm to (83.0, 77.0)
- moved C4 12.1 mm to (83.0, 65.0)
- moved J4 11.7 mm to (106.5, 34.0), turned to 180 degrees
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Routing:
- net GND: track 0.00 -> 274.3 mm, vias 0 -> 1
- net +24V24: track 0.00 -> 188.7 mm
- net Net-(J3-Pin_1): track 0.00 -> 77.9 mm
- net Net-(Q1-G): track 0.00 -> 71.6 mm
- net Net-(D1-A): track 0.00 -> 21.0 mm
- net Net-(J2-Pin_2): track 0.00 -> 17.1 mm
- net Net-(D1-K): track 0.00 -> 14.0 mm
- added copper zone on F.Cu, net +24V24
- added copper zone on B.Cu, net GND
Other:
- board outline added: 84 x 63 mm
