File: Hardware/Horns_v1/Horns_v1.kicad_pcb (KiCad board)
At the start: 2 copper layers, 0 parts

Commit message: firmware error fix and changed hardware connector footprints
Parts:
- added C1: 0.1u, Capacitor_THT:CP_Radial_D5.0mm_P2.00mm, F.Cu at (79.0, 57.0)
- added C2: 0.1u, Capacitor_THT:CP_Radial_D5.0mm_P2.00mm, F.Cu at (104.5, 64.0)
- added C3: 0.1u, Capacitor_THT:CP_Radial_D5.0mm_P2.00mm, F.Cu at (104.5, 71.5)
- added C4: 0.1u, Capacitor_THT:CP_Radial_D5.0mm_P2.00mm, F.Cu at (84.5, 57.0)
- added C5: 1u, Capacitor_THT:CP_Radial_D5.0mm_P2.00mm, F.Cu at (98.0, 57.0)
- added C6: 1u, Capacitor_THT:CP_Radial_D5.0mm_P2.00mm, F.Cu at (98.0, 64.0)
- added C7: 10u, Capacitor_THT:CP_Radial_D5.0mm_P2.00mm, F.Cu at (97.5, 71.5)
- added C8: 10u, Capacitor_THT:CP_Radial_D5.0mm_P2.00mm, F.Cu at (91.0, 57.0)
- added C9: 100u, Capacitor_THT:CP_Radial_D5.0mm_P2.00mm, F.Cu at (93.0, 71.5)
- added D1: US2DA, Diode_SMD:D_SMA, F.Cu at (92.0, 63.5)
- added F1: 2, Fuse:Fuse_0603_1608Metric_Pad1.05x0.95mm_HandSolder, F.Cu at (84.0, 61.0)
- added J5: Conn_01x02, Connector_Molex:Molex_Micro-Fit_3.0_43650-0200_1x02_P3.00mm_Horizontal, F.Cu at (83.0, 76.2)
- added J6: Conn_01x02, Connector_Molex:Molex_Micro-Fit_3.0_43650-0200_1x02_P3.00mm_Horizontal, F.Cu at (80.0, 72.3)
- added J7: Conn_01x02, Connector_Molex:Molex_Micro-Fit_3.0_43650-0200_1x02_P3.00mm_Horizontal, F.Cu at (68.0, 69.5)
- added J8: Conn_01x03, Connector_Molex:Molex_Micro-Fit_3.0_43650-0300_1x03_P3.00mm_Horizontal, F.Cu at (98.0, 76.2)
- added Q1: IRF540N, Package_TO_SOT_THT:TO-220-3_Vertical, F.Cu at (66.9, 76.5)
- added R1: 1k, Resistor_SMD:R_0603_1608Metric_Pad0.98x0.95mm_HandSolder, F.Cu at (78.0, 61.0)
- added REF**: MountingHole_3.2mm_M3, MountingHole:MountingHole_3.2mm_M3, F.Cu at (67.0, 55.0)
- added REF**: MountingHole_3.2mm_M3, MountingHole:MountingHole_3.2mm_M3, F.Cu at (106.0, 55.0)
- added REF**: MountingHole_3.2mm_M3, MountingHole:MountingHole_3.2mm_M3, F.Cu at (67.0, 82.0)
- added REF**: MountingHole_3.2mm_M3, MountingHole:MountingHole_3.2mm_M3, F.Cu at (106.0, 82.0)
Routing:
- net GND: track 0.00 -> 78.7 mm, vias 0 -> 2
- net +24V: track 0.00 -> 60.8 mm
- net Net-(Q1-D): track 0.00 -> 21.2 mm
- net Net-(D1-A): track 0.00 -> 18.4 mm
- net Net-(J6-Pin_2): track 0.00 -> 12.1 mm
- net Net-(J7-Pin_2): track 0.00 -> 11.0 mm
- net /On/Off: track 0.00 -> 7.45 mm
- net Net-(C1-Pad1): track 0.00 -> 4.02 mm
- net Net-(J5-Pin_2): track 0.00 -> 3.86 mm
Other:
- board outline added: 47 x 35 mm
