File: Hardware/Horns_v1/Horns_v1.kicad_sch (KiCad schematic)
At the start: 0 parts

Commit message: firmware error fix and changed hardware connector footprints
Parts:
- added C1, C2, C3, C4: 0.1u, Capacitor_THT:CP_Radial_D5.0mm_P2.00mm, symbol Device:C
- added C5, C6: 1u, Capacitor_THT:CP_Radial_D5.0mm_P2.00mm, symbol Device:C
- added C7, C8: 10u, Capacitor_THT:CP_Radial_D5.0mm_P2.00mm, symbol Device:C
- added C9: 100u, Capacitor_THT:CP_Radial_D5.0mm_P2.00mm, symbol Device:C_Polarized
- added D1: US2DA, Diode_SMD:D_SMA, symbol Diode:US2DA
- added F1: 2, Fuse:Fuse_0603_1608Metric_Pad1.05x0.95mm_HandSolder, symbol device:Fuse
- added J5, J6, J7: Conn_01x02, Connector_Molex:Molex_KK-254_AE-6410-02A_1x02_P2.54mm_Vertical, symbol Connector_Generic:Conn_01x02
- added J8: Conn_01x03, Connector_Molex:Molex_KK-254_AE-6410-03A_1x03_P2.54mm_Vertical, symbol Connector_Generic:Conn_01x03
- added Q1: IRF540N, Package_TO_SOT_THT:TO-220-3_Vertical, symbol Transistor_FET:IRF540N
- added R1: 1k, Resistor_SMD:R_0603_1608Metric_Pad0.98x0.95mm_HandSolder, symbol device:R
Connections:
- new net: F1.2, Q1.2 (D)
- new net: D1.2 (A), J5.1 (Pin_1)
- new net: J5.2 (Pin_2), J6.1 (Pin_1)
- new net: C1.1, R1.2
- new net: F1.1, J6.2 (Pin_2)
- new net: J7.2 (Pin_2), R1.1
- new net +24V: C2.1, C3.1, C4.1, C5.1, C6.1, C7.1, C8.1, C9.1, D1.1 (K), J8.2 (Pin_2)
- new net GND: C1.2, C2.2, C3.2, C4.2, C5.2, C6.2, C7.2, C8.2, C9.2, J8.1 (Pin_1), J8.3 (Pin_3), Q1.3 (S)
- new net On/Off: J7.1 (Pin_1), Q1.1 (G)
Other:
- title: Template -> Horns_Board_V1
