File: Hardware/Dev/Prog1/prog1.kicad_pcb (KiCad board)
At the start: 2 copper layers, 0 parts

Commit message: Firmware Proj 1 & Horns Schematic
Parts:
- added D1: LED_RED, layout:LED_0603_Symbol_on_F.SilkS, F.Cu at (139.0, 103.0)
- added J1: Conn_01x02, Connector_Molex:Molex_KK-254_AE-6410-02A_1x02_P2.54mm_Vertical, F.Cu at (139.7, 108.0)
- added R1: 105, Resistor_SMD:R_0603_1608Metric_Pad0.98x0.95mm_HandSolder, F.Cu at (143.0, 103.0)
- added REF**: MountingHole_3.2mm_M3, MountingHole:MountingHole_3.2mm_M3, F.Cu at (141.0, 96.5)
- added REF**: MountingHole_3.2mm_M3, MountingHole:MountingHole_3.2mm_M3, F.Cu at (148.0, 109.0)
- added SW1: SW_Push, Button_Switch_SMD:SW_DIP_SPSTx01_Slide_6.7x4.1mm_W8.61mm_P2.54mm_LowProfile, F.Cu at (148.0, 97.7)
Routing:
- net Net-(R1-Pad1): track 0.00 -> 12.9 mm
- net GND: track 0.00 -> 2.51 mm, vias 0 -> 1
- net Net-(D1-A): track 0.00 -> 2.29 mm
- added copper zone on F.Cu, net +3V3
- added copper zone on B.Cu, net GND
Other:
- board outline added: 15 x 22 mm
