File: Hardware/LEDProject/LEDProject_v1.kicad_pcb (KiCad board)
At the start: 2 copper layers, 0 parts

Commit message: updated horns board
Parts:
- added D1: LED_RED, layout:LED_0603_Symbol_on_F.SilkS, F.Cu at (111.0, 84.5)
- added J1: Conn_01x02, Connector_Molex:Molex_KK-254_AE-6410-02A_1x02_P2.54mm_Vertical, F.Cu at (114.0, 89.1)
- added R1: 105, Resistor_SMD:R_0603_1608Metric_Pad0.98x0.95mm_HandSolder, F.Cu at (114.6, 84.5)
- added REF**: MountingHole_3.2mm_M3, MountingHole:MountingHole_3.2mm_M3, F.Cu at (112.0, 79.0)
- added REF**: MountingHole_3.2mm_M3, MountingHole:MountingHole_3.2mm_M3, F.Cu at (120.0, 90.0)
- added SW1: SW_Push, Button_Switch_SMD:SW_DIP_SPSTx01_Slide_6.7x4.1mm_W6.73mm_P2.54mm_LowProfile_JPin, F.Cu at (119.0, 80.0)
Routing:
- net Net-(R1-Pad1): track 0.00 -> 10.1 mm
- net GND: track 0.00 -> 2.02 mm, vias 0 -> 1
- net Net-(D1-A): track 0.00 -> 1.85 mm
- added copper zone on F.Cu, net +3V3
- added copper zone on B.Cu, net GND
Other:
- board outline added: 16.1 x 21 mm
