File: Hardware/Dev/ac_Horns_v1.0/ac_Horns_v1.0.kicad_pcb (KiCad board)
At the start: 2 copper layers, 0 parts

Commit message: Horns Project Finish
Parts:
- added C1: 0.1μF, Capacitor_SMD:C_0603_1608Metric, F.Cu at (116.2, 90.5)
- added C2: 0.1uF, Capacitor_SMD:C_0603_1608Metric, F.Cu at (103.0, 91.5)
- added C3: 0.1uF, Capacitor_SMD:C_0603_1608Metric, F.Cu at (103.1, 97.2)
- added C4: 0.1uF, Capacitor_SMD:C_0603_1608Metric, F.Cu at (103.2, 101.4)
- added C5: 1uF, Capacitor_SMD:C_0603_1608Metric, F.Cu at (103.2, 103.2)
- added C6: 1uF, Capacitor_SMD:C_0603_1608Metric, F.Cu at (103.0, 93.5)
- added C7: 10uF, Capacitor_SMD:C_0603_1608Metric, F.Cu at (103.0, 95.2)
- added C8: 10uF, Capacitor_SMD:C_0603_1608Metric, F.Cu at (103.1, 99.3)
- added C9: 100uF, Capacitor_SMD:C_0603_1608Metric, F.Cu at (103.0, 89.7)
- added D1: US2FA, Diode_THT:D_A-405_P10.16mm_Horizontal, F.Cu at (97.0, 91.5)
- added F1: 2A, Fuse:Fuse_0603_1608Metric, F.Cu at (114.0, 101.4)
- added Horn1: Conn_01x02, Connector_Molex:Molex_Micro-Fit_3.0_43650-0200_1x02_P3.00mm_Horizontal, F.Cu at (102.2, 106.6)
- added Horn2: Conn_01x02, Connector_Molex:Molex_Micro-Fit_3.0_43650-0200_1x02_P3.00mm_Horizontal, F.Cu at (114.0, 106.4)
- added J1: Conn_01x03, Connector_Molex:Molex_Micro-Fit_3.0_43650-0300_1x03_P3.00mm_Horizontal, F.Cu at (98.9, 86.8)
- added J2: Conn_01x02, Connector_Molex:Molex_Micro-Fit_3.0_43650-0200_1x02_P3.00mm_Horizontal, F.Cu at (113.3, 86.9)
- added Q1: IRF6727M, Package_DirectFET:DirectFET_MX, F.Cu at (112.8, 95.7)
- added R2: 1k, Resistor_SMD:R_0612_1632Metric, F.Cu at (111.9, 90.7)
- added REF**: MountingHole_3.2mm_M3, MountingHole:MountingHole_3.2mm_M3, F.Cu at (91.0, 113.0)
- added REF**: MountingHole_3.2mm_M3, MountingHole:MountingHole_3.2mm_M3, F.Cu at (91.0, 80.0)
- added REF**: MountingHole_3.2mm_M3, MountingHole:MountingHole_3.2mm_M3, F.Cu at (124.0, 80.0)
- added REF**: MountingHole_3.2mm_M3, MountingHole:MountingHole_3.2mm_M3, F.Cu at (124.0, 113.0)
Routing:
- net GND: track 0.00 -> 45.0 mm, vias 0 -> 2
- net HORN_IN: track 0.00 -> 21.8 mm
- net HornCr: track 0.00 -> 16.8 mm
- net Net-(Q1-D): track 0.00 -> 16.3 mm
- net Net-(Horn1-Pin_1): track 0.00 -> 8.62 mm
- net +24V: track 0.00 -> 6.78 mm
- added copper zone on F.Cu, net +24V
- added copper zone on B.Cu, net GND
Other:
- board outline added: 41 x 41 mm
