File: Hardware/Dev/erickw2_Horns_v0.0/erickw2_Horns_v0.0.kicad_pcb (KiCad board)
At the start: 2 copper layers, 0 parts

Commit message: I have tried my hardest and at this point my circuit looks ok, everything definitely isn't perfect
Parts:
- added C1: 1 microFarad, Capacitor_SMD:CP_Elec_3x5.3, F.Cu at (144.8, 87.9)
- added C2: 1 microFarad, Capacitor_SMD:CP_Elec_3x5.3, F.Cu at (119.9, 94.0)
- added C3: 1 microFarad, Capacitor_SMD:CP_Elec_3x5.3, F.Cu at (138.7, 94.0)
- added C4: 0.1 microF, Capacitor_SMD:CP_Elec_3x5.3, F.Cu at (114.8, 94.0)
- added C5: 0.1 microF, Capacitor_SMD:CP_Elec_3x5.3, F.Cu at (125.0, 94.0)
- added C6: 0.1 microF, Capacitor_SMD:CP_Elec_3x5.3, F.Cu at (134.1, 94.0)
- added C7: 10 microF, Capacitor_SMD:CP_Elec_3x5.3, F.Cu at (109.7, 94.0)
- added C8: 10 microF, Capacitor_SMD:CP_Elec_3x5.3, F.Cu at (129.5, 94.0)
- added C9: 100 microF, Capacitor_SMD:CP_Elec_3x5.3, F.Cu at (143.3, 94.0)
- added D1: 1N4148WT, Diode_SMD:D_SOD-523, F.Cu at (120.7, 71.1)
- added F1: 2A, Fuse:Fuse_Bourns_MF-RG300, F.Cu at (131.1, 70.5)
- added J1: Conn_01x02, Connector_Molex:Molex_Micro-Fit_3.0_43650-0210_1x02-1MP_P3.00mm_Horizontal, F.Cu at (146.3, 71.6)
- added J2: Conn_01x02, Connector_Molex:Molex_Micro-Fit_3.0_43650-0210_1x02-1MP_P3.00mm_Horizontal, F.Cu at (114.3, 81.8)
- added J3: Conn_01x03, Connector_Molex:Molex_Micro-Fit_3.0_43650-0300_1x03_P3.00mm_Horizontal, F.Cu at (105.2, 95.3)
- added J4: Conn_01x02, Connector_Molex:Molex_Micro-Fit_3.0_43650-0210_1x02-1MP_P3.00mm_Horizontal, F.Cu at (126.5, 81.8)
- added Q1: IRLZ44N, Package_TO_SOT_THT:TO-220-3_Vertical, F.Cu at (135.5, 79.1)
- added R1: 1 KOhm, Resistor_SMD:R_0201_0603Metric, F.Cu at (141.5, 80.8)
- added REF**: Horn Control, TerminalBlock_Altech:Altech_AK300_1x02_P5.00mm_45-Degree, F.Cu at (151.6, 88.3)
- added REF**: MountingHole_3.2mm_M3, MountingHole:MountingHole_3.2mm_M3, F.Cu at (99.6, 69.1)
- added REF**: MountingHole_3.2mm_M3, MountingHole:MountingHole_3.2mm_M3, F.Cu at (156.0, 69.1)
- added REF**: MountingHole_3.2mm_M3, MountingHole:MountingHole_3.2mm_M3, F.Cu at (156.0, 103.1)
- added REF**: MountingHole_3.2mm_M3, MountingHole:MountingHole_3.2mm_M3, F.Cu at (99.6, 103.1)
Routing:
- net GND: track 0.00 -> 98.0 mm
- net +24V: track 0.00 -> 65.4 mm
- net /Horn Control: track 0.00 -> 41.9 mm
- net Net-(D1-A): track 0.00 -> 16.4 mm
- net Net-(Q1-D): track 0.00 -> 11.3 mm
- net Net-(J2-Pin_1): track 0.00 -> 9.19 mm
- net Net-(Q1-G): track 0.00 -> 6.40 mm
- added copper zone on F.Cu, net +24V
- added copper zone on B.Cu, net GND
Other:
- board outline added: 68.6 x 46.7 mm
