File: Hardware/ProjectTwo (Horns Board)/ProjectTwo.kicad_pcb (KiCad board)
At the start: 2 copper layers, 0 parts

Commit message: Finished horns board schematic
Parts:
- added C1: 0.1uF, Capacitor_SMD:C_1206_3216Metric, F.Cu at (132.0, 84.0)
- added C2: 0.1uF, Capacitor_SMD:C_1206_3216Metric, F.Cu at (132.0, 88.0)
- added C3: 0.1uF, Capacitor_SMD:C_1206_3216Metric, F.Cu at (132.0, 92.0)
- added C4: 1uF, Capacitor_SMD:C_1206_3216Metric, F.Cu at (132.0, 96.0)
- added C5: 1uF, Capacitor_SMD:C_1206_3216Metric, F.Cu at (132.0, 100.0)
- added C6: 10uF, Capacitor_SMD:C_1206_3216Metric, F.Cu at (132.0, 104.0)
- added C7: 10uF, Capacitor_SMD:C_1206_3216Metric, F.Cu at (132.0, 108.0)
- added CC1: 0.1uF, Capacitor_SMD:C_1206_3216Metric, F.Cu at (150.0, 102.0)
- added D1: DioideRectifier, Diode_SMD:D_SMA, F.Cu at (139.0, 85.0)
- added F1: 2A, Fuse:Fuse_1206_3216Metric, F.Cu at (150.0, 96.0)
- added F2: 2A, Fuse:Fuse_1206_3216Metric, F.Cu at (146.0, 85.0)
- added Horn1: Conn_01x02_Pin, TerminalBlock:TerminalBlock_bornier-2_P5.08mm, F.Cu at (139.5, 103.0)
- added Horn2: Conn_01x02_Pin, TerminalBlock:TerminalBlock_bornier-2_P5.08mm, F.Cu at (139.5, 93.0)
- added HornControl1: Conn_01x02_Pin, TerminalBlock:TerminalBlock_bornier-2_P5.08mm, F.Cu at (142.0, 111.5)
- added PolarizedC1: 100uF, Capacitor_THT:CP_Radial_D6.3mm_P2.50mm, F.Cu at (133.0, 114.0)
- added Power1: Conn_01x03_Pin, TerminalBlock:TerminalBlock_bornier-3_P5.08mm, F.Cu at (125.0, 104.1)
- added Q1: AO3400A, Package_TO_SOT_SMD:SOT-23, F.Cu at (151.0, 90.0)
- added R1: 1000, Resistor_SMD:R_0805_2012Metric, F.Cu at (150.0, 107.0)
- added REF**: MountingHole_3.2mm_M3, MountingHole:MountingHole_3.2mm_M3, F.Cu at (125.0, 86.0)
- added REF**: MountingHole_3.2mm_M3, MountingHole:MountingHole_3.2mm_M3, F.Cu at (150.0, 115.0)
Routing:
- net Net-(D1-A): track 0.00 -> 101.8 mm
- net /24 V: track 0.00 -> 73.2 mm
- net Net-(Horn1-Pin_2): track 0.00 -> 19.5 mm
- net GND: track 0.00 -> 15.5 mm, vias 0 -> 4
- net Net-(Horn1-Pin_1): track 0.00 -> 10.0 mm
- net Net-(D1-K): track 0.00 -> 9.47 mm
- net /Horn Control Net: track 0.00 -> 8.93 mm
- net Net-(Q1-D): track 0.00 -> 6.10 mm
- net Net-(Q1-G): track 0.00 -> 4.45 mm
- net Net-(CC1-Pad1): track 0.00 -> 3.90 mm
- net Net-(CC1-Pad2): track 0.00 -> 3.12 mm
- added copper zone on F.Cu, net /24 V
- added copper zone on B.Cu, net GND
Other:
- board outline added: 37 x 41 mm
