File: Hardware/hengrun2_Horns_v1.0/Template_Horns_v1.0/hengrun2_horns_v1.0.kicad_sch (KiCad schematic)
At the start: 0 parts

Commit message: finished horn schematic
Parts:
- added C1: 0.1uF, Capacitor_SMD:C_0603_1608Metric, symbol device:C
- added C2, C3, C4: 0.1uF, Capacitor_SMD:C_0603_1608Metric, symbol device:C_Small
- added C5, C6: 1uF, Capacitor_SMD:C_0603_1608Metric, symbol device:C_Small
- added C7, C8: 10uF, Capacitor_SMD:C_0603_1608Metric, symbol device:C_Small
- added C9: 100uF, Capacitor_THT:CP_Radial_D5.0mm_P2.50mm, symbol Device:C_Polarized_Small
- added D1: ES2DA-13-F, Diode_SMD:D_SMA, symbol Device:D
- added F1, F2: 2A, Fuse:Fuse_1206_3216Metric, symbol device:Fuse
- added J1: Conn_01x03, Connector_Molex:Molex_KK-254_AE-6410-03A_1x03_P2.54mm_Vertical, symbol Connector_Generic:Conn_01x03
- added J2, J3, J4: Conn_01x02, Connector_Molex:Molex_KK-254_AE-6410-02A_1x02_P2.54mm_Vertical, symbol Connector_Generic:Conn_01x02
- added Q1: IRLZ44N, Package_TO_SOT_THT:TO-220-3_Vertical, symbol Transistor_FET:IRLZ44N
- added R1: 1kΩ, Resistor_SMD:R_0603_1608Metric_Pad0.98x0.95mm_HandSolder, symbol device:R_US
Connections:
- new net: F1.2, Q1.2 (D)
- new net: C1.2, R1.1
- new net: J2.2 (Pin_2), R1.2
- new net: F2.2, Q1.1 (G)
- new net +24V: C2.1, C3.1, C4.1, C5.1, C6.1, C7.1, C8.1, C9.1, D1.1 (K), J1.2 (Pin_2), J3.1 (Pin_1)
- new net GND: C1.1, C2.2, C3.2, C4.2, C5.2, C6.2, C7.2, C8.2, C9.2, J1.1 (Pin_1), J1.3 (Pin_3), Q1.3 (S)
- new net HORN_CTL: F2.1, J2.1 (Pin_1)
- new net HORN_IN: D1.2 (A), F1.1, J4.2 (Pin_2)
- new net HORN_OUT: J3.2 (Pin_2), J4.1 (Pin_1)
Other:
- title: Template -> hengrun2_horn
