File: Hardware/hengrun2_Horns_v1.0/Template_Horns_v1.0/hengrun2_horns_v1.0.kicad_pcb (KiCad board)
At the start: 2 copper layers, 0 parts

Commit message: finished horn PCB
Parts:
- added C1: 0.1uF, Capacitor_SMD:C_0603_1608Metric, F.Cu at (151.2, 101.0)
- added C2: 0.1uF, Capacitor_SMD:C_0603_1608Metric, F.Cu at (142.4, 78.0)
- added C3: 0.1uF, Capacitor_SMD:C_0603_1608Metric, F.Cu at (142.4, 81.0)
- added C4: 0.1uF, Capacitor_SMD:C_0603_1608Metric, F.Cu at (142.4, 84.0)
- added C5: 1uF, Capacitor_SMD:C_0603_1608Metric, F.Cu at (142.4, 87.0)
- added C6: 1uF, Capacitor_SMD:C_0603_1608Metric, F.Cu at (142.2, 90.0)
- added C7: 10uF, Capacitor_SMD:C_0603_1608Metric, F.Cu at (142.2, 93.0)
- added C8: 10uF, Capacitor_SMD:C_0603_1608Metric, F.Cu at (142.4, 96.0)
- added C9: 100uF, Capacitor_THT:CP_Radial_D5.0mm_P2.50mm, F.Cu at (141.5, 101.0)
- added D1: ES2DA-13-F, Diode_SMD:D_SMA, F.Cu at (157.0, 85.0)
- added F1: 2A, Fuse:Fuse_1206_3216Metric, F.Cu at (168.6, 78.0)
- added F2: 2A, Fuse:Fuse_1206_3216Metric, F.Cu at (164.0, 95.0)
- added J1: Conn_01x03, Connector_Molex:Molex_KK-254_AE-6410-03A_1x03_P2.54mm_Vertical, F.Cu at (150.9, 94.0)
- added J2: Conn_01x02, Connector_Molex:Molex_KK-254_AE-6410-02A_1x02_P2.54mm_Vertical, F.Cu at (165.0, 101.0)
- added J3: Conn_01x02, Connector_Molex:Molex_KK-254_AE-6410-02A_1x02_P2.54mm_Vertical, F.Cu at (150.5, 76.0)
- added J4: Conn_01x02, Connector_Molex:Molex_KK-254_AE-6410-02A_1x02_P2.54mm_Vertical, F.Cu at (159.5, 76.0)
- added Q1: IRLZ44N, Package_TO_SOT_THT:TO-220-3_Vertical, F.Cu at (170.0, 90.1)
- added R1: 1kΩ, Resistor_SMD:R_0603_1608Metric_Pad0.98x0.95mm_HandSolder, F.Cu at (156.9, 101.0)
- added REF**: MountingHole_3.2mm_M3, MountingHole:MountingHole_3.2mm_M3, F.Cu at (140.0, 70.0)
- added REF**: MountingHole_3.2mm_M3, MountingHole:MountingHole_3.2mm_M3, F.Cu at (173.0, 110.0)
- added REF**: MountingHole_3.2mm_M3, MountingHole:MountingHole_3.2mm_M3, F.Cu at (173.0, 70.0)
- added REF**: MountingHole_3.2mm_M3, MountingHole:MountingHole_3.2mm_M3, F.Cu at (140.0, 110.0)
Routing:
- net +24V: track 0.00 -> 70.8 mm
- net GND: track 0.00 -> 33.5 mm, vias 0 -> 2
- net Net-(Q1-D): track 0.00 -> 19.5 mm
- net /HORN_IN: track 0.00 -> 16.9 mm
- net Net-(Q1-G): track 0.00 -> 9.52 mm
- net /HORN_CTL: track 0.00 -> 7.23 mm
- net /HORN_OUT: track 0.00 -> 6.46 mm
- net Net-(J2-Pin_2): track 0.00 -> 4.64 mm
- net Net-(C1-Pad2): track 0.00 -> 4.00 mm
- added copper zone on F.Cu, net +24V
- added copper zone on B.Cu, net GND
Other:
- board outline added: 41 x 48 mm
