File: Hardware/HornsBoard_v0.0/HornsBoard_v0.0.kicad_sch (KiCad schematic)
At the start: 0 parts

Commit message: horns schematic done
Parts:
- added C1, C2, C3, C4: 0.1 uF, symbol Device:C
- added C5, C6: 1 uF, symbol Device:C
- added C7, C8: 10 uF, symbol Device:C
- added C9: 100 uF, symbol Device:C_Polarized_US
- added D1: 1N4001, Diode_THT:D_DO-41_SOD81_P10.16mm_Horizontal, symbol Diode:1N4001
- added F1: 2A, symbol device:Fuse
- added J1, J2, J4: Conn_01x02, symbol Connector_Generic:Conn_01x02
- added J3: Conn_01x03, symbol Connector_Generic:Conn_01x03
- added Q1: IRF9383M, Package_DirectFET:DirectFET_MX, symbol Transistor_FET:IRF9383M
- added R1: 1K Ohms, symbol device:R
Connections:
- new net: F1.1, Q1.1 (D)
- new net: F1.2, J1.2 (Pin_2)
- new net: J1.1 (Pin_1), J2.2 (Pin_2)
- new net +24V: D1.2 (A)
- new net GND: C1.2, C2.1, C2.2, C3.1, C3.2, C4.1, C4.2, C5.1, C5.2, C6.1, C6.2, C7.1, C7.2, C8.1, C8.2, C9.1, C9.2, D1.1 (K), J2.1 (Pin_1), J3.1 (Pin_1), J3.2 (Pin_2), J3.3 (Pin_3), J4.1 (Pin_1), Q1.3 (S), R1.2
- new net HORN_CONTROL: C1.1, J4.2 (Pin_2), Q1.2 (G), R1.1
