File: Hardware/odommom2_horns_v1.0/odommom2_horns_v1.0.kicad_sch (KiCad schematic)
At the start: 0 parts

Commit message: horns board complete + dfm
Parts:
- added C1, C2: 0.1µF, Capacitor_SMD:C_0603_1608Metric_Pad1.08x0.95mm_HandSolder, symbol Device:C
- added C3, C4: 0.1µF, Capacitor_SMD:C_0603_1608Metric_Pad1.08x0.95mm_HandSolder, symbol device:C
- added C5, C6: 1µF, Capacitor_SMD:C_0603_1608Metric_Pad1.08x0.95mm_HandSolder, symbol device:C
- added C7, C8: 10µF, Capacitor_SMD:C_0603_1608Metric_Pad1.08x0.95mm_HandSolder, symbol device:C
- added C9: 100µF, Capacitor_SMD:C_0603_1608Metric_Pad1.08x0.95mm_HandSolder, symbol device:C_Polarized
- added D1: US2DA, Diode_SMD:D_SMA, symbol Diode:US2DA
- added F1: 2A, Fuse:Fuse_0603_1608Metric_Pad1.05x0.95mm_HandSolder, symbol Device:Fuse
- added J1: Conn_01x03, Connector_Molex:Molex_KK-254_AE-6410-03A_1x03_P2.54mm_Vertical, symbol Connector_Generic:Conn_01x03
- added J2, J3, J4: Conn_01x02, Connector_Molex:Molex_KK-254_AE-6410-02A_1x02_P2.54mm_Vertical, symbol Connector_Generic:Conn_01x02
- added Q1: BSS138, Package_TO_SOT_SMD:SOT-23, symbol Transistor_FET:BSS138
- added R1: 1000Ω, Resistor_SMD:R_0603_1608Metric_Pad0.98x0.95mm_HandSolder, symbol Device:R
Connections:
- new net: F1.1, Q1.2 (S)
- new net: J3.1 (Pin_1), J4.2 (Pin_2)
- new net +24V: C2.1, C3.1, C4.1, C5.1, C6.1, C7.1, C8.1, C9.1, D1.1 (K)
- new net GND: C1.1, C2.2, C3.2, C4.2, C5.2, C6.2, C7.2, C8.2, C9.2, J1.1 (Pin_1), J1.3 (Pin_3), J2.2 (Pin_2), J3.2 (Pin_2), Q1.3 (D), R1.1
- new net HORN_CTRL: C1.2, J2.1 (Pin_1), Q1.1 (G), R1.2
- new net HORN_IN: D1.2 (A), F1.2, J4.1 (Pin_1)
