File: Hardware/hejmadi2_Horns_v1.0/Horns_Board_v0.0.kicad_pcb (KiCad board)
At the start: 2 copper layers, 0 parts

Commit message: Horns Board pcb
Parts:
- added C1: 0.1µF, Capacitor_SMD:C_0603_1608Metric_Pad1.08x0.95mm_HandSolder, F.Cu at (122.7, 94.0)
- added C2: 0.1µF, Capacitor_SMD:C_0603_1608Metric_Pad1.08x0.95mm_HandSolder, F.Cu at (122.7, 96.5)
- added C3: 0.1µF, Capacitor_SMD:C_0603_1608Metric_Pad1.08x0.95mm_HandSolder, F.Cu at (122.7, 99.0)
- added C4: 0.1µF, Capacitor_SMD:C_0603_1608Metric_Pad1.08x0.95mm_HandSolder, F.Cu at (122.7, 101.5)
- added C5: 1uF, Capacitor_SMD:C_0603_1608Metric_Pad1.08x0.95mm_HandSolder, F.Cu at (122.7, 104.0)
- added C6: 1uF, Capacitor_SMD:C_0603_1608Metric_Pad1.08x0.95mm_HandSolder, F.Cu at (122.7, 106.0)
- added C7: 10uF, Capacitor_SMD:C_0603_1608Metric_Pad1.08x0.95mm_HandSolder, F.Cu at (127.1, 94.0)
- added C8: 10uF, Capacitor_SMD:C_0603_1608Metric_Pad1.08x0.95mm_HandSolder, F.Cu at (127.1, 96.5)
- added C9: 100uF, Capacitor_SMD:C_0603_1608Metric_Pad1.08x0.95mm_HandSolder, F.Cu at (127.1, 99.0)
- added D1: US2DA, Diode_SMD:D_SMA, F.Cu at (149.5, 101.5)
- added F1: 2A, Fuse:Fuse_0603_1608Metric_Pad1.05x0.95mm_HandSolder, F.Cu at (126.2, 103.0)
- added J1: Conn_01x03, Connector_Molex:Molex_Micro-Fit_3.0_43650-0300_1x03_P3.00mm_Horizontal, F.Cu at (134.2, 106.1)
- added J2: Conn_01x02, Connector_Molex:Molex_Micro-Fit_3.0_43650-0200_1x02_P3.00mm_Horizontal, F.Cu at (133.0, 94.6)
- added J3: Conn_01x02, Connector_Molex:Molex_Micro-Fit_3.0_43650-0200_1x02_P3.00mm_Horizontal, F.Cu at (144.2, 94.6)
- added J4: Conn_01x02, Connector_Molex:Molex_Micro-Fit_3.0_43650-0200_1x02_P3.00mm_Horizontal, F.Cu at (155.6, 97.6)
- added Q1: IRFR010PBF, Package_SON:Fairchild_DualPower33-6_3x3mm, F.Cu at (149.4, 106.0)
- added R1: 1k, Resistor_SMD:R_0603_1608Metric_Pad0.98x0.95mm_HandSolder, F.Cu at (129.2, 102.2)
- added REF**: MountingHole_3.2mm_M3, MountingHole:MountingHole_3.2mm_M3, F.Cu at (159.0, 105.0)
- added REF**: MountingHole_3.2mm_M3, MountingHole:MountingHole_3.2mm_M3, F.Cu at (124.0, 89.0)
Routing:
- net /HORN_IN: track 0.00 -> 85.6 mm
- net Net-(C1-Pad1): track 0.00 -> 38.7 mm
- net /HORN_CTL: track 0.00 -> 32.6 mm
- net Net-(Q1-D): track 0.00 -> 32.3 mm
- net GND: track 0.00 -> 29.7 mm, vias 0 -> 2
- net Net-(D1-A): track 0.00 -> 17.0 mm
- net Net-(D1-K): track 0.00 -> 14.3 mm
- added copper zone on F.Cu, net +24V
- added copper zone on B.Cu, net GND
Other:
- board outline added: 43 x 24 mm
