File: Hardware/prog2_Horns_v1.0/prog2_Horns_v1.0.kicad_pcb (KiCad board)
At the start: 2 copper layers, 0 parts

Commit message: Horns project PCB complete
Parts:
- added C1: 0.1uf, layout:CP_Oval_L16.0mm_W8.0mm_P11.5mm, F.Cu at (62.5, 119.5)
- added C2: C_Small, layout:CP_Oval_L16.0mm_W8.0mm_P11.5mm, F.Cu at (53.5, 142.0)
- added C3: 0.1uF, layout:CP_Oval_L16.0mm_W8.0mm_P11.5mm, F.Cu at (70.8, 142.0)
- added C4: 0.1uF, layout:CP_Oval_L16.0mm_W8.0mm_P11.5mm, F.Cu at (87.8, 142.0)
- added C5: 1uF, layout:CP_Oval_L16.0mm_W8.0mm_P11.5mm, F.Cu at (104.8, 142.0)
- added C6: 1uF, layout:CP_Oval_L16.0mm_W8.0mm_P11.5mm, F.Cu at (53.8, 155.5)
- added C7: 10uF, layout:CP_Oval_L16.0mm_W8.0mm_P11.5mm, F.Cu at (70.8, 155.5)
- added C8: 0.1uF, layout:CP_Oval_L16.0mm_W8.0mm_P11.5mm, F.Cu at (105.2, 154.5)
- added C9: 100uF, layout:CP_Radial_D16.5mm_P5.08mm, F.Cu at (85.4, 158.5)
- added D1: US2AA, Diode_SMD:D_SMA, F.Cu at (83.0, 128.5)
- added F1: 2A, layout:Fuse_Littelfuse_1206, F.Cu at (92.6, 121.5)
- added F2: 2A, layout:Fuse_Littelfuse_1206, F.Cu at (86.1, 119.0)
- added F3: 2A, layout:Fuse_Littelfuse_1206, F.Cu at (121.0, 131.4)
- added HORN_CTL1: Conn_01x02, Connector_Molex:Molex_CLIK-Mate_502382-0270_1x02-1MP_P1.25mm_Vertical, F.Cu at (81.9, 114.5)
- added HORN_IN1: Conn_01x02, Connector_Molex:Molex_CLIK-Mate_502382-0270_1x02-1MP_P1.25mm_Vertical, F.Cu at (122.1, 140.0)
- added HORN_OUT1: Conn_01x02, Connector_Molex:Molex_CLIK-Mate_502382-0270_1x02-1MP_P1.25mm_Vertical, F.Cu at (122.1, 152.0)
- added J1: Conn_01x03, Connector_Molex:Molex_CLIK-Mate_502382-0370_1x03-1MP_P1.25mm_Vertical, F.Cu at (42.0, 129.8)
- added Q1: Q_PMOS_SGD, Package_DirectFET:DirectFET_L4, F.Cu at (114.0, 123.2)
- added R1: 1k, Resistor_SMD:R_0805_2012Metric_Pad1.20x1.40mm_HandSolder, F.Cu at (50.1, 120.0)
- added REF**: MountingHole, MountingHole:MountingHole_3.2mm_M3, F.Cu at (126.0, 113.5)
- added REF**: MountingHole, MountingHole:MountingHole_3.2mm_M3, F.Cu at (126.5, 168.0)
- added REF**: MountingHole, MountingHole:MountingHole_3.2mm_M3, F.Cu at (40.5, 167.0)
- added REF**: MountingHole, MountingHole:MountingHole_3.2mm_M3, F.Cu at (40.0, 113.5)
Routing:
- net GND: track 0.00 -> 234.7 mm, vias 0 -> 2
- net +24V: track 0.00 -> 229.6 mm
- net /source: track 0.00 -> 74.9 mm
- net Net-(D1-K): track 0.00 -> 39.7 mm
- net Net-(HORN_CTL1-Pin_1): track 0.00 -> 38.0 mm
- net /gate: track 0.00 -> 27.2 mm
- net Net-(HORN_IN1-Pin_2): track 0.00 -> 19.8 mm
- net /Drain: track 0.00 -> 14.1 mm
- net Net-(C1-Pad1): track 0.00 -> 7.19 mm
- net /horn_control: track 0.00 -> 3.41 mm
- added copper zone on F.Cu, net +24V
- added copper zone on B.Cu, net GND
Other:
- board outline added: 96 x 64 mm
