File: Hardware/ali79_Horns_v2.0/horns_v2.kicad_pcb (KiCad board)
At the start: 2 copper layers, 35 x 30 mm, 19 parts, among them J1 Conn_01x03, J2 Conn_01x02, J3 Conn_01x02, J4 Conn_01x02, Q1 IRF6646

Commit message: Applied changes to the diode
Connections:
- J3 pad 1: Net-(D1-A) -> Net-(D1-K)
- J4 pad 2: Net-(D1-K) -> Net-(D1-A)
Routing:
- net Net-(D1-K): track 10.9 -> 5.30 mm
Changed lines of the file:
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@@
 			(layers "*.Cu" "*.Mask")
 			(remove_unused_layers no)
-			(net 7 "Net-(D1-K)")
+			(net 1 "Net-(D1-A)")
 			(pinfunction "Pin_2")
 			(pintype "passive")
@@
 		(tags "Diode SMA (DO-214AC)")
 		(property "Reference" "D1"
-			(at 0 -2.5 360)
+			(at 0 -2.5 0)
 			(layer "F.SilkS")
 			(effects
@@
 		)
 		(property "Value" "Rectifier Diode"
-			(at 0 2.6 360)
+			(at 0 2.6 0)
 			(layer "F.Fab")
 			(hide yes)
@@
 		)
 		(property "Footprint" "Diode_SMD:D_SMA"
-			(at 0 0 360)
+			(at 0 0 0)
 			(layer "F.Fab")
 			(hide yes)
@@
 		)
 		(property "Datasheet" "https://www.diodes.com/assets/Datasheets/ds14002.pdf"
-			(at 0 0 360)
+			(at 0 0 0)
 			(layer "F.Fab")
 			(hide yes)
@@
 		)
 		(property "Description" "200V, 1.5A, General Purpose Rectifier Diode, SMA(DO-214AC)"
-			(at 0 0 360)
+			(at 0 0 0)
 			(layer "F.Fab")
 			(hide yes)
@@
 		)
 		(fp_text user "${REFERENCE}"
-			(at 0 -2.5 360)
+			(at 0 -2.5 0)
 			(layer "F.Fab")
 			(effects
@@
 		(tags "connector Molex Micro-Fit_3.0 top entry")
 		(property "Reference" "J3"
-			(at 1.5 -10.32 360)
+			(at 1.5 -10.32 0)
 			(layer "F.SilkS")
 			(effects
@@
 		)
 		(property "Value" "Conn_01x02"
-			(at -2.5 -13.32 360)
+			(at -2.5 -13.32 0)
 			(layer "F.Fab")
 			(hide yes)
@@
 		)
 		(property "Footprint" "Connector_Molex:Molex_Micro-Fit_3.0_43650-0200_1x02_P3.00mm_Horizontal"
-			(at 0 0 360)
+			(at 0 0 0)
 			(layer "F.Fab")
 			(hide yes)
@@
 		)
 		(property "Datasheet" ""
-			(at 0 0 360)
+			(at 0 0 0)
 			(layer "F.Fab")
 			(hide yes)
@@
 		)
 		(property "Description" "Generic connector, single row, 01x02, script generated (kicad-library-utils/schlib/autogen/connector/)"
-			(at 0 0 360)
+			(at 0 0 0)
 			(layer "F.Fab")
 			(hide yes)
@@
 			(remove_unused_layers no)
 			(roundrect_rratio 0.166667)
-			(net 1 "Net-(D1-A)")
+			(net 7 "Net-(D1-K)")
 			(pinfunction "Pin_1")
 			(pintype "passive")
@@
 	)
 	(segment
-		(start 119.5 54)
-		(end 121 54)
+		(start 115.5 49.5)
+		(end 115.5 47.97)
 		(width 0.25)
 		(layer "F.Cu")
@@
 	)
 	(segment
-		(start 119 53.5)
-		(end 119.5 54)
+		(start 118.5 50)
+		(end 116 50)
 		(width 0.25)
 		(layer "F.Cu")
@@
 	)
 	(segment
-		(start 119 52)
-		(end 119 53.5)
+		(start 116 50)
+		(end 115.5 49.5)
 		(width 0.25)
 		(layer "F.Cu")
@@
 	)
 	(segment
-		(start 121.5 54.5)
-		(end 121.5 56.68)
+		(start 119 52)
+		(end 119 50.5)
 		(width 0.25)
 		(layer "F.Cu")
@@
 	)
 	(segment
-		(start 121 54)
-		(end 121.5 54.5)
+		(start 119 50.5)
+		(end 118.5 50)
 		(width 0.25)
 		(layer "F.Cu")
@@
 	)
 	(segment
-		(start 123 50.5)
-		(end 123 52)
-		(width 0.25)
-		(layer "F.Cu")
-		(net 7)
-	)
-	(segment
-		(start 115.5 49.5)
-		(end 116 50)
-		(width 0.25)
-		(layer "F.Cu")
-		(net 7)
-	)
-	(segment
-		(start 116 50)
-		(end 122.5 50)
+		(start 123 53.5)
+		(end 121.5 55)
 		(width 0.25)
 		(layer "F.Cu")
@@
 	)
 	(segment
-		(start 122.5 50)
-		(end 123 50.5)
+		(start 123 52)
+		(end 123 53.5)
 		(width 0.25)
 		(layer "F.Cu")
@@
 	)
 	(segment
-		(start 115.5 47.97)
-		(end 115.5 49.5)
+		(start 121.5 55)
+		(end 121.5 56.68)
 		(width 0.25)
 		(layer "F.Cu")
