File: Hardware/Dev/Template_v0.0/Template_v0.0.kicad_pcb (KiCad board)
At the start: 2 copper layers, 0 parts

Commit message: easy hardware and easy/hard firmware
Parts:
- added D1: LED_RED, layout:LED_0603_Symbol_on_F.SilkS, F.Cu at (126.4, 113.0)
- added J1: Conn_01x02, Connector_Molex:Molex_KK-254_AE-6410-02A_1x02_P2.54mm_Vertical, F.Cu at (129.7, 119.3)
- added R2: 105, Resistor_SMD:R_0603_1608Metric_Pad0.98x0.95mm_HandSolder, F.Cu at (130.1, 112.9)
- added REF**: MountingHole_3.2mm_M3, MountingHole:MountingHole_3.2mm_M3, F.Cu at (137.5, 118.7)
- added REF**: MountingHole_3.2mm_M3, MountingHole:MountingHole_3.2mm_M3, F.Cu at (130.0, 107.3)
- added SW1: SW_Push, Button_Switch_SMD:SW_DIP_SPSTx01_Slide_6.7x4.1mm_W8.61mm_P2.54mm_LowProfile, F.Cu at (136.5, 108.5)
Routing:
- net Net-(R2-Pad1): track 0.00 -> 12.0 mm
- net GND: track 0.00 -> 5.37 mm, vias 0 -> 1
- net Net-(D1-A): track 0.00 -> 2.03 mm
- added copper zone on F.Cu, net +3V3
- added copper zone on B.Cu, net GND
Other:
- board outline added: 18.9 x 25.1 mm
